File: smd_aio.sch (KiCad schematic (older format))
At the start: 4 parts, among them SW1 SW_PUSH

Commit message: newer
Parts:
- added C10, C3, C4, C6, C8, C9: 100n, symbol C
- added C2, C5, C7: 10u, symbol CP
- added Q5: FZT751TA, symbol Q_PNP_BCE
- added R6: 1K, symbol R
Connections:
- wire segments 17 -> 49
Other:
- note added: "<1% tolerance"
- moved on the sheet: C1, R1, SW1, U?

Commit message: DSP angeschlossen
Parts:
- added C12, C15: 10u, symbol C
- added C13, C16, C17: 100n, symbol C
- added C14: 10u, symbol CP
- added C18: 3n3, symbol C
- added C19: 56n, symbol C
- added R11: 475, symbol R
- added R8: 18K, symbol R
Connections:
- net +3V3: now also U?.38 (PLL_MODE0), U?.39 (PLL_MODE1), C18.1, R11.1
- net GND: now also U?.30 (RSVD), C12.2, C13.2, C14.2, C15.2, C16.2, C17.2, R8.2
- net ADC0: now reaches U?.2 (ADC0)
- net ADC0: now also U?.4 (ADC1)
- net at U?.3 (ADC_RES): now also R8.1
- net MCLK0: now reaches U?.32 (MCLKI)
- net at U?.35 (PLL_LF): now also C18.2, C19.2
- net at U?.40 (CM): now also C14.1, C16.1
- net at U?.41 (FILTD): now also C15.1, C17.1
- net VOUT3: now reaches U?.43 (VOUT3)
- net VOUT3: now also U?.44 (VOUT2), U?.45 (VOUT1), U?.46 (VOUT0)
- net at U?.47 (FILTA): now also C12.1, C13.1
- new net: C19.1, R11.2
- no-connect marks 0 -> 1
