File: SOURCES/clock.sch (KiCad schematic (older format))
At the start: 6 parts, among them X1 Crystal_Oszillator

Commit message: design rule check
Parts:
- gave numbers to parts that had none: 2
- renumbered C70 to C89, C71 to C90, FB5 to FB3
Changed lines of the file:
@@
 LIBS:fdsp_transistor_new
 LIBS:LM2738XMY&slash_NOPB-symbols
-LIBS:smd_aio-cache
 EELAYER 25 0
 EELAYER END
@@
 $EndComp
 $Comp
-L FILTER FB5
+L FILTER FB3
 U 1 1 5B0715ED
 P 3050 2560
-F 0 "FB5" H 3050 2710 50  0000 C CNN
+F 0 "FB3" H 3050 2710 50  0000 C CNN
 F 1 "330" H 3050 2460 50  0000 C CNN
 F 2 "" H 3050 2560 50  0000 C CNN
@@
 $EndComp
 $Comp
-L +3V3 #PWR109
+L +3V3 #PWR0130
 U 1 1 5B071680
 P 3050 1930
-F 0 "#PWR109" H 3050 1780 50  0001 C CNN
+F 0 "#PWR0130" H 3050 1780 50  0001 C CNN
 F 1 "+3V3" H 3050 2070 50  0000 C CNN
 F 2 "" H 3050 1930 60  0000 C CNN
@@
 $EndComp
 $Comp
-L C C70
+L C C89
 U 1 1 5B0716DF
 P 3050 3270
-F 0 "C70" H 3075 3370 50  0000 L CNN
+F 0 "C89" H 3075 3370 50  0000 L CNN
 F 1 "10u" H 3075 3170 50  0000 L CNN
 F 2 "" H 3088 3120 30  0000 C CNN
@@
 $EndComp
 $Comp
-L GND #PWR110
+L GND #PWR0131
 U 1 1 5B071722
 P 3050 3850
-F 0 "#PWR110" H 3050 3600 50  0001 C CNN
+F 0 "#PWR0131" H 3050 3600 50  0001 C CNN
 F 1 "GND" H 3050 3700 50  0000 C CNN
 F 2 "" H 3050 3850 60  0000 C CNN
@@
 MCLK5
 $Comp
-L C C71
+L C C90
 U 1 1 5B07311B
 P 6020 3580
-F 0 "C71" H 6045 3680 50  0000 L CNN
+F 0 "C90" H 6045 3680 50  0000 L CNN
 F 1 "100n" H 6045 3480 50  0000 L CNN
 F 2 "" H 6058 3430 30  0000 C CNN
@@
 $EndComp
 $Comp
-L GND #PWR111
+L GND #PWR0132
 U 1 1 5B0732C4
 P 6020 3870
-F 0 "#PWR111" H 6020 3620 50  0001 C CNN
+F 0 "#PWR0132" H 6020 3620 50  0001 C CNN
 F 1 "GND" H 6020 3720 50  0000 C CNN
 F 2 "" H 6020 3870 60  0000 C CNN
@@
 MCLK4
 $Comp
-L IDT2309NZ U?
+L IDT2309NZ U10
 U 1 1 5B108D74
 P 6910 3040
-F 0 "U?" H 6710 3490 60  0000 C CNN
+F 0 "U10" H 6710 3490 60  0000 C CNN
 F 1 "IDT2309NZ" H 6960 2290 60  0000 C CNN
 F 2 "" H 6910 2690 60  0001 C CNN
@@
 Connection ~ 6020 2940
 $Comp
-L R R?
+L R R40
 U 1 1 5B1890A3
 P 7910 3040
-F 0 "R?" V 7990 3040 50  0000 C CNN
+F 0 "R40" V 7990 3040 50  0000 C CNN
 F 1 "24" V 7910 3040 50  0000 C CNN
 F 2 "" V 7840 3040 30  0000 C CNN
