File: SOURCES/clock.sch (KiCad schematic (older format))
At the start: 12 parts, among them P22 TST, U10 IDT2309NZ, X1 ASV-24.576MHz-EJ-T

Commit message: started layout
Parts:
- added P28, P29, P30: TST, fdsp_misc:Measurement_Point_Round-SMD-Pad_Small, symbol TST
Connections:
- net at U10.14 (OUTPUT7): now also P30.1
- net at U10.15 (OUTPUT8): now also P29.1
- net at U10.16 (OUTPUT9): now also P28.1
- no-connect marks 3 -> 0
Changed lines of the file:
@@
 $EndComp
 $Comp
-L +3V3 #PWR0137
+L +3V3 #PWR0138
 U 1 1 5B071680
 P 3050 1930
-F 0 "#PWR0137" H 3050 1780 50  0001 C CNN
+F 0 "#PWR0138" H 3050 1780 50  0001 C CNN
 F 1 "+3V3" H 3050 2070 50  0000 C CNN
 F 2 "" H 3050 1930 60  0000 C CNN
@@
 $EndComp
 $Comp
-L GND #PWR0138
+L GND #PWR0139
 U 1 1 5B071722
 P 3050 3850
-F 0 "#PWR0138" H 3050 3600 50  0001 C CNN
+F 0 "#PWR0139" H 3050 3600 50  0001 C CNN
 F 1 "GND" H 3050 3700 50  0000 C CNN
 F 2 "" H 3050 3850 60  0000 C CNN
@@
 $EndComp
 $Comp
-L GND #PWR0139
+L GND #PWR0140
 U 1 1 5B0732C4
 P 6020 3870
-F 0 "#PWR0139" H 6020 3620 50  0001 C CNN
+F 0 "#PWR0140" H 6020 3620 50  0001 C CNN
 F 1 "GND" H 6020 3720 50  0000 C CNN
 F 2 "" H 6020 3870 60  0000 C CNN
@@
 Text GLabel 8160 3140 2    60   Output ~ 0
 MCLK4
+Connection ~ 3050 2940
+Wire Wire Line
+	3050 3420 3050 3850
+Wire Wire Line
+	3050 2910 3050 3120
+Wire Wire Line
+	3050 1930 3050 2210
+Wire Wire Line
+	3990 3650 3050 3650
+Connection ~ 3050 3650
+Wire Wire Line
+	3950 2940 3950 3150
+Wire Wire Line
+	3950 3150 3990 3150
+Connection ~ 3950 2940
+Wire Wire Line
+	5090 3150 5260 3150
+Wire Wire Line
+	5260 3150 5260 2940
+Connection ~ 5260 2940
+Wire Wire Line
+	5090 3650 5810 3650
+Wire Wire Line
+	5810 3650 5810 3240
+Wire Wire Line
+	5810 3240 6460 3240
+Wire Wire Line
+	6020 3730 6020 3870
+Wire Wire Line
+	6460 3790 6020 3790
+Wire Wire Line
+	6460 3490 6460 3790
+Connection ~ 6020 3790
+Connection ~ 6460 3690
+Connection ~ 6460 3590
+Wire Wire Line
+	3050 2940 6460 2940
+Wire Wire Line
+	6430 2740 6430 2940
+Wire Wire Line
+	6430 2840 6460 2840
+Connection ~ 6430 2940
+Wire Wire Line
+	6430 2740 6460 2740
+Connection ~ 6430 2840
+Wire Wire Line
+	6020 3430 6020 2940
+Connection ~ 6020 2940
+$Comp
+L R R45
+U 1 1 5B1890A3
+P 7910 3040
+F 0 "R45" V 7990 3040 50  0000 C CNN
+F 1 "34" V 7910 3040 50  0000 C CNN
+F 2 "fdsp_resistor:R_1206_HandSoldering" V 7840 3040 30  0001 C CNN
+F 3 "" H 7910 3040 30  0000 C CNN
+	1    7910 3040
+	0    1    1    0
+$EndComp
+Wire Wire Line
+	7460 3040 7760 3040
+Wire Wire Line
+	8060 3040 8160 3040
+$Comp
+L R R40
+U 1 1 5B1F732A
+P 7665 2940
+F 0 "R40" V 7745 2940 50  0000 C CNN
+F 1 "34" V 7665 2940 50  0000 C CNN
+F 2 "fdsp_resistor:R_1206_HandSoldering" V 7595 2940 30  0001 C CNN
+F 3 "" H 7665 2940 30  0000 C CNN
+	1    7665 2940
+	0    1    1    0
+$EndComp
+Wire Wire Line
+	7460 2940 7515 2940
+Wire Wire Line
+	7815 2940 8160 2940
+$Comp
+L R R44
+U 1 1 5B1F742C
+P 7910 2840
+F 0 "R44" V 7990 2840 50  0000 C CNN
+F 1 "34" V 7910 2840 50  0000 C CNN
+F 2 "fdsp_resistor:R_1206_HandSoldering" V 7840 2840 30  0001 C CNN
+F 3 "" H 7910 2840 30  0000 C CNN
+	1    7910 2840
+	0    1    1    0
+$EndComp
+$Comp
+L R R43
+U 1 1 5B1F7478
+P 7670 2740
+F 0 "R43" V 7750 2740 50  0000 C CNN
+F 1 "34" V 7670 2740 50  0000 C CNN
+F 2 "fdsp_resistor:R_1206_HandSoldering" V 7600 2740 30  0001 C CNN
+F 3 "" H 7670 2740 30  0000 C CNN
+	1    7670 2740
+	0    1    1    0
+$EndComp
+Wire Wire Line
+	7460 2740 7520 2740
+Wire Wire Line
+	7820 2740 8160 2740
+Wire Wire Line
+	8160 2740 8160 2735
+Wire Wire Line
+	7460 2840 7760 2840
+Wire Wire Line
+	8060 2840 8160 2840
+$Comp
+L R R41
+U 1 1 5B1F76D9
+P 7665 3140
+F 0 "R41" V 7745 3140 50  0000 C CNN
+F 1 "34" V 7665 3140 50  0000 C CNN
+F 2 "fdsp_resistor:R_1206_HandSoldering" V 7595 3140 30  0001 C CNN
+F 3 "" H 7665 3140 30  0000 C CNN
+	1    7665 3140
+	0    1    1    0
+$EndComp
+Wire Wire Line
+	7460 3140 7515 3140
+Wire Wire Line
+	7815 3140 8160 3140
+$Comp
+L R R42
+U 1 1 5B1F7927
+P 7665 3340
+F 0 "R42" V 7745 3340 50  0000 C CNN
+F 1 "34" V 7665 3340 50  0000 C CNN
+F 2 "fdsp_resistor:R_1206_HandSoldering" V 7595 3340 30  0001 C CNN
+F 3 "" H 7665 3340 30  0000 C CNN
+	1    7665 3340
+	0    1    1    0
+$EndComp
+Wire Wire Line
+	7460 3340 7515 3340
+Wire Wire Line
+	7815 3340 8160 3340
+Wire Wire Line
+	8160 3340 8160 3335
+$Comp
+L TST P22
+U 1 1 5B219E4B
+P 5405 3550
+F 0 "P22" H 5405 3850 50  0000 C BNN
+F 1 "TST" H 5405 3800 50  0000 C CNN
+F 2 "fdsp_misc:Measurement_Point_Round-SMD-Pad_Small" H 5405 3550 50  0001 C CNN
+F 3 "" H 5405 3550 50  0000 C CNN
+	1    5405 3550
+	1    0    0    -1
+$EndComp
+Wire Wire Line
+	5405 3550 5405 3650
+Connection ~ 5405 3650
 $Comp
 L IDT2309NZ U10
@@
 	1    0    0    -1
 $EndComp
-NoConn ~ 7460 3440
-NoConn ~ 7460 3540
-NoConn ~ 7460 3640
-Connection ~ 3050 2940
-Wire Wire Line
-	3050 3420 3050 3850
-Wire Wire Line
-	3050 2910 3050 3120
-Wire Wire Line
-	3050 1930 3050 2210
-Wire Wire Line
-	3990 3650 3050 3650
-Connection ~ 3050 3650
-Wire Wire Line
-	3950 2940 3950 3150
-Wire Wire Line
-	3950 3150 3990 3150
-Connection ~ 3950 2940
-Wire Wire Line
-	5090 3150 5260 3150
-Wire Wire Line
-	5260 3150 5260 2940
-Connection ~ 5260 2940
-Wire Wire Line
-	5090 3650 5810 3650
-Wire Wire Line
-	5810 3650 5810 3240
-Wire Wire Line
-	5810 3240 6460 3240
-Wire Wire Line
-	6020 3730 6020 3870
-Wire Wire Line
-	6460 3790 6020 3790
-Wire Wire Line
-	6460 3490 6460 3790
-Connection ~ 6020 3790
-Connection ~ 6460 3690
-Connection ~ 6460 3590
-Wire Wire Line
-	3050 2940 6460 2940
-Wire Wire Line
-	6430 2740 6430 2940
-Wire Wire Line
-	6430 2840 6460 2840
-Connection ~ 6430 2940
-Wire Wire Line
-	6430 2740 6460 2740
-Connection ~ 6430 2840
-Wire Wire Line
-	6020 3430 6020 2940
-Connection ~ 6020 2940
-$Comp
-L R R45
-U 1 1 5B1890A3
-P 7910 3040
-F 0 "R45" V 7990 3040 50  0000 C CNN
-F 1 "34" V 7910 3040 50  0000 C CNN
-F 2 "fdsp_resistor:R_1206_HandSoldering" V 7840 3040 30  0001 C CNN
-F 3 "" H 7910 3040 30  0000 C CNN
-	1    7910 3040
-	0    1    1    0
-$EndComp
-Wire Wire Line
-	7460 3040 7760 3040
-Wire Wire Line
-	8060 3040 8160 3040
-$Comp
-L R R40
-U 1 1 5B1F732A
-P 7665 2940
-F 0 "R40" V 7745 2940 50  0000 C CNN
-F 1 "34" V 7665 2940 50  0000 C CNN
-F 2 "fdsp_resistor:R_1206_HandSoldering" V 7595 2940 30  0001 C CNN
-F 3 "" H 7665 2940 30  0000 C CNN
-	1    7665 2940
-	0    1    1    0
-$EndComp
-Wire Wire Line
-	7460 2940 7515 2940
-Wire Wire Line
-	7815 2940 8160 2940
-$Comp
-L R R44
-U 1 1 5B1F742C
-P 7910 2840
-F 0 "R44" V 7990 2840 50  0000 C CNN
-F 1 "34" V 7910 2840 50  0000 C CNN
-F 2 "fdsp_resistor:R_1206_HandSoldering" V 7840 2840 30  0001 C CNN
-F 3 "" H 7910 2840 30  0000 C CNN
-	1    7910 2840
-	0    1    1    0
-$EndComp
-$Comp
-L R R43
-U 1 1 5B1F7478
-P 7670 2740
-F 0 "R43" V 7750 2740 50  0000 C CNN
-F 1 "34" V 7670 2740 50  0000 C CNN
-F 2 "fdsp_resistor:R_1206_HandSoldering" V 7600 2740 30  0001 C CNN
-F 3 "" H 7670 2740 30  0000 C CNN
-	1    7670 2740
-	0    1    1    0
-$EndComp
-Wire Wire Line
-	7460 2740 7520 2740
-Wire Wire Line
-	7820 2740 8160 2740
-Wire Wire Line
-	8160 2740 8160 2735
-Wire Wire Line
-	7460 2840 7760 2840
-Wire Wire Line
-	8060 2840 8160 2840
-$Comp
-L R R41
-U 1 1 5B1F76D9
-P 7665 3140
-F 0 "R41" V 7745 3140 50  0000 C CNN
-F 1 "34" V 7665 3140 50  0000 C CNN
-F 2 "fdsp_resistor:R_1206_HandSoldering" V 7595 3140 30  0001 C CNN
-F 3 "" H 7665 3140 30  0000 C CNN
-	1    7665 3140
-	0    1    1    0
-$EndComp
-Wire Wire Line
-	7460 3140 7515 3140
-Wire Wire Line
-	7815 3140 8160 3140
-$Comp
-L R R42
-U 1 1 5B1F7927
-P 7665 3340
-F 0 "R42" V 7745 3340 50  0000 C CNN
-F 1 "34" V 7665 3340 50  0000 C CNN
-F 2 "fdsp_resistor:R_1206_HandSoldering" V 7595 3340 30  0001 C CNN
-F 3 "" H 7665 3340 30  0000 C CNN
-	1    7665 3340
-	0    1    1    0
-$EndComp
-Wire Wire Line
-	7460 3340 7515 3340
-Wire Wire Line
-	7815 3340 8160 3340
-Wire Wire Line
-	8160 3340 8160 3335
-$Comp
-L TST P22
-U 1 1 5B219E4B
-P 5405 3550
-F 0 "P22" H 5405 3850 50  0000 C BNN
-F 1 "TST" H 5405 3800 50  0000 C CNN
-F 2 "fdsp_misc:Measurement_Point_Round-SMD-Pad_Small" H 5405 3550 50  0001 C CNN
-F 3 "" H 5405 3550 50  0000 C CNN
-	1    5405 3550
-	1    0    0    -1
-$EndComp
-Wire Wire Line
-	5405 3550 5405 3650
-Connection ~ 5405 3650
+$Comp
+L TST P30
+U 1 1 5B23DE97
+P 7805 3485
+F 0 "P30" H 7805 3785 50  0000 C BNN
+F 1 "TST" H 7805 3735 50  0000 C CNN
+F 2 "fdsp_misc:Measurement_Point_Round-SMD-Pad_Small" H 7805 3485 50  0001 C CNN
+F 3 "" H 7805 3485 50  0000 C CNN
+	1    7805 3485
+	0    1    1    0
+$EndComp
+$Comp
+L TST P29
+U 1 1 5B23DFA7
+P 7705 3640
+F 0 "P29" H 7705 3940 50  0000 C BNN
+F 1 "TST" H 7705 3890 50  0000 C CNN
+F 2 "fdsp_misc:Measurement_Point_Round-SMD-Pad_Small" H 7705 3640 50  0001 C CNN
+F 3 "" H 7705 3640 50  0000 C CNN
+	1    7705 3640
+	0    1    1    0
+$EndComp
+$Comp
+L TST P28
+U 1 1 5B23E075
+P 7580 3775
+F 0 "P28" H 7580 4075 50  0000 C BNN
+F 1 "TST" H 7580 4025 50  0000 C CNN
+F 2 "fdsp_misc:Measurement_Point_Round-SMD-Pad_Small" H 7580 3775 50  0001 C CNN
+F 3 "" H 7580 3775 50  0000 C CNN
+	1    7580 3775
+	0    1    1    0
+$EndComp
+Wire Wire Line
+	7460 3440 7460 3485
+Wire Wire Line
+	7460 3485 7805 3485
+Wire Wire Line
+	7460 3540 7705 3540
+Wire Wire Line
+	7705 3540 7705 3640
+Wire Wire Line
+	7460 3640 7580 3640
+Wire Wire Line
+	7580 3640 7580 3775
 $EndSCHEMATC
