File: SOURCES/SPDIFin.sch (KiCad schematic (older format))
At the start: 17 parts, among them U6 CS8422-CNZ

Commit message: design rule check
Parts:
- gave numbers to parts that had none: 15
- renumbered C72 to C46, U6 to U5
Connections:
- wire segments 51 -> 60
Changed lines of the file:
@@
 LIBS:fdsp_transistor_new
 LIBS:LM2738XMY&slash_NOPB-symbols
-LIBS:smd_aio-cache
 EELAYER 25 0
 EELAYER END
@@
 $EndDescr
 $Comp
-L CS8422-CNZ U6
+L CS8422-CNZ U5
 U 1 1 5B04A0D3
-P 4290 3150
-F 0 "U6" H 5790 3550 60  0000 C CNN
-F 1 "CS8422-CNZ" H 5790 3450 60  0000 C CNN
-F 2 "CIR-QFN-32_5X5" H 5790 3390 60  0001 C CNN
-F 3 "" H 4290 3150 60  0000 C CNN
-	1    4290 3150
+P 4300 3150
+F 0 "U5" H 5800 3550 60  0000 C CNN
+F 1 "CS8422-CNZ" H 5800 3450 60  0000 C CNN
+F 2 "CIR-QFN-32_5X5" H 5800 3390 60  0001 C CNN
+F 3 "" H 4300 3150 60  0000 C CNN
+	1    4300 3150
 	1    0    0    -1
 $EndComp
@@
 SPDIF_In
 $Comp
-L GND #PWR?
+L GND #PWR065
 U 1 1 5B0AA933
 P 4100 3600
-F 0 "#PWR?" H 4100 3350 50  0001 C CNN
+F 0 "#PWR065" H 4100 3350 50  0001 C CNN
 F 1 "GND" H 4100 3450 50  0000 C CNN
 F 2 "" H 4100 3600 60  0000 C CNN
@@
 $EndComp
 $Comp
-L GND #PWR?
+L GND #PWR066
 U 1 1 5B0AAA5E
 P 4100 4100
-F 0 "#PWR?" H 4100 3850 50  0001 C CNN
+F 0 "#PWR066" H 4100 3850 50  0001 C CNN
 F 1 "GND" V 4100 3900 50  0000 C CNN
 F 2 "" H 4100 4100 60  0000 C CNN
@@
 BRD_RST
 $Comp
-L C C72
+L C C46
 U 1 1 5B0AB301
 P 3400 3250
-F 0 "C72" V 3350 3300 50  0000 L CNN
+F 0 "C46" V 3350 3300 50  0000 L CNN
 F 1 "10n" V 3350 3050 50  0000 L CNN
 F 2 "" H 3438 3100 30  0000 C CNN
@@
 $EndComp
 $Comp
-L GND #PWR?
+L GND #PWR067
 U 1 1 5B0ABCD3
 P 3150 3250
-F 0 "#PWR?" H 3150 3000 50  0001 C CNN
+F 0 "#PWR067" H 3150 3000 50  0001 C CNN
 F 1 "GND" V 3150 3050 50  0000 C CNN
 F 2 "" H 3150 3250 60  0000 C CNN
@@
 $EndComp
 $Comp
-L GND #PWR?
+L GND #PWR068
 U 1 1 5B0AC2AB
 P 4100 3450
-F 0 "#PWR?" H 4100 3200 50  0001 C CNN
+F 0 "#PWR068" H 4100 3200 50  0001 C CNN
 F 1 "GND" H 4100 3300 50  0000 C CNN
 F 2 "" H 4100 3450 60  0000 C CNN
@@
 NoConn ~ 5300 3350
 $Comp
-L GND #PWR?
+L GND #PWR069
 U 1 1 5B0AC367
 P 4100 4350
-F 0 "#PWR?" H 4100 4100 50  0001 C CNN
+F 0 "#PWR069" H 4100 4100 50  0001 C CNN
 F 1 "GND" V 4100 4150 50  0000 C CNN
 F 2 "" H 4100 4350 60  0000 C CNN
@@
 	4150 4150 4300 4150
 Wire Wire Line
-	4150 4050 4150 4150
+	4150 4050 4150 4100
+Wire Wire Line
+	4150 4100 4150 4150
 Wire Wire Line
 	4300 4050 4150 4050
@@
 	4150 3650 4300 3650
 Wire Wire Line
-	4150 3550 4150 3650
+	4150 3550 4150 3600
+Wire Wire Line
+	4150 3600 4150 3650
 Wire Wire Line
 	4300 3550 4150 3550
 $Comp
-L C C?
+L C C43
 U 1 1 5B0AC50B
 P 2750 4400
-F 0 "C?" H 2650 4500 50  0000 L CNN
+F 0 "C43" H 2650 4500 50  0000 L CNN
 F 1 "100n" H 2550 4300 50  0000 L CNN
 F 2 "" H 2788 4250 30  0000 C CNN
@@
 $EndComp
 $Comp
-L CP C?
+L CP C45
 U 1 1 5B0AC538
 P 3050 4400
-F 0 "C?" H 3075 4500 50  0000 L CNN
+F 0 "C45" H 3075 4500 50  0000 L CNN
 F 1 "10µ" H 3075 4300 50  0000 L CNN
 F 2 "" H 3088 4250 30  0000 C CNN
@@
 $EndComp
 $Comp
-L GND #PWR?
+L GND #PWR070
 U 1 1 5B0AC5D5
 P 2900 4650
-F 0 "#PWR?" H 2900 4400 50  0001 C CNN
+F 0 "#PWR070" H 2900 4400 50  0001 C CNN
 F 1 "GND" H 2900 4500 50  0000 C CNN
 F 2 "" H 2900 4650 60  0000 C CNN
@@
 $EndComp
 Wire Wire Line
-	2750 4250 4300 4250
+	2750 4250 3050 4250
+Wire Wire Line
+	3050 4250 4300 4250
 Connection ~ 3050 4250
 Wire Wire Line
 	2750 4550 2750 4600
 Wire Wire Line
-	2750 4600 3050 4600
+	2750 4600 2900 4600
+Wire Wire Line
+	2900 4600 3050 4600
 Wire Wire Line
 	2900 4600 2900 4650
@@
 Connection ~ 2900 4600
 $Comp
-L C C?
+L C C48
 U 1 1 5B0AC750
 P 8450 4400
-F 0 "C?" H 8475 4500 50  0000 L CNN
+F 0 "C48" H 8475 4500 50  0000 L CNN
 F 1 "100n" H 8475 4300 50  0000 L CNN
 F 2 "" H 8488 4250 30  0000 C CNN
@@
 $EndComp
 $Comp
-L CP C?
+L CP C49
 U 1 1 5B0AC756
 P 8750 4400
-F 0 "C?" H 8775 4500 50  0000 L CNN
+F 0 "C49" H 8775 4500 50  0000 L CNN
 F 1 "10µ" H 8775 4300 50  0000 L CNN
 F 2 "" H 8788 4250 30  0000 C CNN
@@
 $EndComp
 $Comp
-L GND #PWR?
+L GND #PWR071
 U 1 1 5B0AC75C
 P 8600 4650
-F 0 "#PWR?" H 8600 4400 50  0001 C CNN
+F 0 "#PWR071" H 8600 4400 50  0001 C CNN
 F 1 "GND" H 8600 4500 50  0000 C CNN
 F 2 "" H 8600 4650 60  0000 C CNN
@@
 	8450 4550 8450 4600
 Wire Wire Line
-	8450 4600 8750 4600
+	8450 4600 8600 4600
+Wire Wire Line
+	8600 4600 8750 4600
 Wire Wire Line
 	8600 4600 8600 4650
@@
 Connection ~ 8600 4600
 Wire Wire Line
-	7300 4250 8750 4250
+	7300 4250 8450 4250
+Wire Wire Line
+	8450 4250 8750 4250
 Connection ~ 8450 4250
 $Comp
-L +3V3 #PWR?
+L +3V3 #PWR072
 U 1 1 5B0AC84E
 P 3050 4250
-F 0 "#PWR?" H 3050 4100 50  0001 C CNN
+F 0 "#PWR072" H 3050 4100 50  0001 C CNN
 F 1 "+3V3" H 3150 4350 50  0000 C CNN
 F 2 "" H 3050 4250 60  0000 C CNN
@@
 	7300 3450 7750 3450
 $Comp
-L LED D?
+L LED D4
 U 1 1 5B0AD170
 P 8800 3350
-F 0 "D?" H 8800 3450 50  0000 C CNN
+F 0 "D4" H 8800 3450 50  0000 C CNN
 F 1 "LED" H 8800 3250 50  0000 C CNN
 F 2 "" H 8800 3350 60  0000 C CNN
@@
 $EndComp
 $Comp
-L R R?
+L R R29
 U 1 1 5B0AD1B9
 P 8250 3350
-F 0 "R?" V 8330 3350 50  0000 C CNN
+F 0 "R29" V 8330 3350 50  0000 C CNN
 F 1 "1k" V 8250 3350 50  0000 C CNN
 F 2 "" V 8180 3350 30  0000 C CNN
@@
 	8400 3350 8600 3350
 $Comp
-L GND #PWR?
+L GND #PWR073
 U 1 1 5B0AD2EA
 P 9200 3350
-F 0 "#PWR?" H 9200 3100 50  0001 C CNN
+F 0 "#PWR073" H 9200 3100 50  0001 C CNN
 F 1 "GND" V 9200 3150 50  0000 C CNN
 F 2 "" H 9200 3350 60  0000 C CNN
@@
 	9000 3350 9200 3350
 $Comp
-L GND #PWR?
+L GND #PWR074
 U 1 1 5B0AD75F
 P 7450 4150
-F 0 "#PWR?" H 7450 3900 50  0001 C CNN
+F 0 "#PWR074" H 7450 3900 50  0001 C CNN
 F 1 "GND" V 7450 3950 50  0000 C CNN
 F 2 "" H 7450 4150 60  0000 C CNN
@@
 	7300 4150 7450 4150
 $Comp
-L C C?
+L C C47
 U 1 1 5B0AD7AE
 P 7950 4050
-F 0 "C?" V 7900 4150 50  0000 L CNN
+F 0 "C47" V 7900 4150 50  0000 L CNN
 F 1 "100n" V 7900 3800 50  0000 L CNN
 F 2 "" H 7988 3900 30  0000 C CNN
@@
 $EndComp
 $Comp
-L GND #PWR?
+L GND #PWR075
 U 1 1 5B0AD8E4
 P 8250 4050
-F 0 "#PWR?" H 8250 3800 50  0001 C CNN
+F 0 "#PWR075" H 8250 3800 50  0001 C CNN
 F 1 "GND" V 8250 3850 50  0000 C CNN
 F 2 "" H 8250 4050 60  0000 C CNN
@@
 NoConn ~ 7300 4550
 $Comp
-L R R?
+L R R27
 U 1 1 5B0AD987
 P 7700 4450
-F 0 "R?" V 7780 4450 50  0000 C CNN
+F 0 "R27" V 7780 4450 50  0000 C CNN
 F 1 "20k" V 7700 4450 50  0000 C CNN
 F 2 "" V 7630 4450 30  0000 C CNN
@@
 $EndComp
 $Comp
-L +3V3 #PWR?
+L +3V3 #PWR076
 U 1 1 5B0ADA22
 P 7950 4450
-F 0 "#PWR?" H 7950 4300 50  0001 C CNN
+F 0 "#PWR076" H 7950 4300 50  0001 C CNN
 F 1 "+3V3" V 7950 4590 50  0000 C CNN
 F 2 "" H 7950 4450 60  0000 C CNN
@@
 NoConn ~ 7300 3150
 $Comp
-L C C?
+L C C42
 U 1 1 5B0ADBB9
 P 2750 3500
-F 0 "C?" H 2650 3600 50  0000 L CNN
+F 0 "C42" H 2650 3600 50  0000 L CNN
 F 1 "100n" H 2550 3400 50  0000 L CNN
 F 2 "" H 2788 3350 30  0000 C CNN
@@
 $EndComp
 $Comp
-L CP C?
+L CP C44
 U 1 1 5B0ADBBF
 P 3050 3500
-F 0 "C?" H 3075 3600 50  0000 L CNN
+F 0 "C44" H 3075 3600 50  0000 L CNN
 F 1 "10µ" H 3075 3400 50  0000 L CNN
 F 2 "" H 3088 3350 30  0000 C CNN
@@
 $EndComp
 $Comp
-L GND #PWR?
+L GND #PWR077
 U 1 1 5B0ADBC5
 P 2900 3750
-F 0 "#PWR?" H 2900 3500 50  0001 C CNN
+F 0 "#PWR077" H 2900 3500 50  0001 C CNN
 F 1 "GND" H 2900 3600 50  0000 C CNN
 F 2 "" H 2900 3750 60  0000 C CNN
@@
 $EndComp
 Wire Wire Line
-	2750 3350 4300 3350
+	2750 3350 3050 3350
+Wire Wire Line
+	3050 3350 4300 3350
 Connection ~ 3050 3350
 Wire Wire Line
 	2750 3650 2750 3700
 Wire Wire Line
-	2750 3700 3050 3700
+	2750 3700 2900 3700
+Wire Wire Line
+	2900 3700 3050 3700
 Wire Wire Line
 	2900 3700 2900 3750
@@
 Connection ~ 2900 3700
 $Comp
-L +3V3 #PWR?
+L +3V3 #PWR078
 U 1 1 5B0ADBD2
 P 2750 3350
-F 0 "#PWR?" H 2750 3200 50  0001 C CNN
+F 0 "#PWR078" H 2750 3200 50  0001 C CNN
 F 1 "+3V3" H 2600 3450 50  0000 C CNN
 F 2 "" H 2750 3350 60  0000 C CNN
@@
 Connection ~ 2750 3350
 $Comp
-L R R?
+L R R25
 U 1 1 5B0ADE1F
 P 3650 3750
-F 0 "R?" V 3730 3750 50  0000 C CNN
+F 0 "R25" V 3730 3750 50  0000 C CNN
 F 1 "32k4" V 3650 3750 50  0000 C CNN
 F 2 "" V 3580 3750 30  0000 C CNN
@@
 $EndComp
 $Comp
-L R R?
+L R R26
 U 1 1 5B0ADF07
 P 3650 3850
-F 0 "R?" V 3550 3850 50  0000 C CNN
+F 0 "R26" V 3550 3850 50  0000 C CNN
 F 1 "16k2" V 3650 3850 50  0000 C CNN
 F 2 "" V 3580 3850 30  0000 C CNN
@@
 	4300 3750 3800 3750
 $Comp
-L GND #PWR?
+L GND #PWR079
 U 1 1 5B0AE249
 P 3450 3800
-F 0 "#PWR?" H 3450 3550 50  0001 C CNN
+F 0 "#PWR079" H 3450 3550 50  0001 C CNN
 F 1 "GND" V 3450 3600 50  0000 C CNN
 F 2 "" H 3450 3800 60  0000 C CNN
@@
 	3500 3750 3450 3750
 Wire Wire Line
-	3450 3750 3450 3850
+	3450 3750 3450 3800
+Wire Wire Line
+	3450 3800 3450 3850
 Wire Wire Line
 	3450 3850 3500 3850
 Connection ~ 3450 3800
 $Comp
-L R R?
+L R R28
 U 1 1 5B0AE799
 P 7700 4650
-F 0 "R?" V 7780 4650 50  0000 C CNN
+F 0 "R28" V 7780 4650 50  0000 C CNN
 F 1 "20k" V 7700 4650 50  0000 C CNN
 F 2 "" V 7630 4650 30  0000 C CNN
@@
 $EndComp
 $Comp
-L +3V3 #PWR?
+L +3V3 #PWR080
 U 1 1 5B0AE79F
 P 7950 4650
-F 0 "#PWR?" H 7950 4500 50  0001 C CNN
+F 0 "#PWR080" H 7950 4500 50  0001 C CNN
 F 1 "+3V3" V 7950 4790 50  0000 C CNN
 F 2 "" H 7950 4650 60  0000 C CNN
@@
 	3150 3250 3250 3250
 $Comp
-L LED D?
+L LED D5
 U 1 1 5B178F6E
 P 8800 4850
-F 0 "D?" H 8800 4950 50  0000 C CNN
+F 0 "D5" H 8800 4950 50  0000 C CNN
 F 1 "LED" H 8800 4750 50  0000 C CNN
 F 2 "" H 8800 4850 60  0000 C CNN
@@
 $EndComp
 $Comp
-L R R?
+L R R30
 U 1 1 5B178F74
 P 8250 4850
-F 0 "R?" V 8330 4850 50  0000 C CNN
+F 0 "R30" V 8330 4850 50  0000 C CNN
 F 1 "1k" V 8250 4850 50  0000 C CNN
 F 2 "" V 8180 4850 30  0000 C CNN
@@
 	8400 4850 8600 4850
 $Comp
-L GND #PWR?
+L GND #PWR081
 U 1 1 5B178F7C
 P 9200 4850
-F 0 "#PWR?" H 9200 4600 50  0001 C CNN
+F 0 "#PWR081" H 9200 4600 50  0001 C CNN
 F 1 "GND" V 9200 4650 50  0000 C CNN
 F 2 "" H 9200 4850 60  0000 C CNN

Commit message: design rule check
Connections:
- net at U5.10 (V/*AUDIO): no longer R30.2
- net at U5.9 (NV/RERR): now also R30.2
- net SPDIF_In renamed SPDIF_IN
- no-connect marks 11 -> 10
Other:
- moved on the sheet: D5, R30
Changed lines of the file:
@@
 LIBS:fdsp_transistor_new
 LIBS:LM2738XMY&slash_NOPB-symbols
+LIBS:smd_aio-cache
 EELAYER 25 0
 EELAYER END
@@
 $EndComp
 Text GLabel 4100 3150 0    60   Input ~ 0
-SPDIF_In
+SPDIF_IN
 $Comp
 L GND #PWR065
@@
 	0    1    1    0
 $EndComp
-NoConn ~ 7300 4950
 NoConn ~ 7300 4850
 NoConn ~ 7300 4350
@@
 	4150 4150 4300 4150
 Wire Wire Line
-	4150 4050 4150 4100
-Wire Wire Line
-	4150 4100 4150 4150
+	4150 4050 4150 4150
 Wire Wire Line
 	4300 4050 4150 4050
@@
 	4150 3650 4300 3650
 Wire Wire Line
-	4150 3550 4150 3600
-Wire Wire Line
-	4150 3600 4150 3650
+	4150 3550 4150 3650
 Wire Wire Line
 	4300 3550 4150 3550
@@
 $EndComp
 Wire Wire Line
-	2750 4250 3050 4250
-Wire Wire Line
-	3050 4250 4300 4250
+	2750 4250 4300 4250
 Connection ~ 3050 4250
 Wire Wire Line
 	2750 4550 2750 4600
 Wire Wire Line
-	2750 4600 2900 4600
-Wire Wire Line
-	2900 4600 3050 4600
+	2750 4600 3050 4600
 Wire Wire Line
 	2900 4600 2900 4650
@@
 	8450 4550 8450 4600
 Wire Wire Line
-	8450 4600 8600 4600
-Wire Wire Line
-	8600 4600 8750 4600
+	8450 4600 8750 4600
 Wire Wire Line
 	8600 4600 8600 4650
@@
 Connection ~ 8600 4600
 Wire Wire Line
-	7300 4250 8450 4250
-Wire Wire Line
-	8450 4250 8750 4250
+	7300 4250 8750 4250
 Connection ~ 8450 4250
 $Comp
@@
 $EndComp
 Wire Wire Line
-	2750 3350 3050 3350
-Wire Wire Line
-	3050 3350 4300 3350
+	2750 3350 4300 3350
 Connection ~ 3050 3350
 Wire Wire Line
 	2750 3650 2750 3700
 Wire Wire Line
-	2750 3700 2900 3700
-Wire Wire Line
-	2900 3700 3050 3700
+	2750 3700 3050 3700
 Wire Wire Line
 	2900 3700 2900 3750
@@
 	3500 3750 3450 3750
 Wire Wire Line
-	3450 3750 3450 3800
-Wire Wire Line
-	3450 3800 3450 3850
+	3450 3750 3450 3850
 Wire Wire Line
 	3450 3850 3500 3850
@@
 L LED D5
 U 1 1 5B178F6E
-P 8800 4850
-F 0 "D5" H 8800 4950 50  0000 C CNN
-F 1 "LED" H 8800 4750 50  0000 C CNN
-F 2 "" H 8800 4850 60  0000 C CNN
-F 3 "" H 8800 4850 60  0000 C CNN
-	1    8800 4850
+P 8800 4950
+F 0 "D5" H 8800 5050 50  0000 C CNN
+F 1 "LED" H 8800 4850 50  0000 C CNN
+F 2 "" H 8800 4950 60  0000 C CNN
+F 3 "" H 8800 4950 60  0000 C CNN
+	1    8800 4950
 	-1   0    0    1
 $EndComp
@@
 L R R30
 U 1 1 5B178F74
-P 8250 4850
-F 0 "R30" V 8330 4850 50  0000 C CNN
-F 1 "1k" V 8250 4850 50  0000 C CNN
-F 2 "" V 8180 4850 30  0000 C CNN
-F 3 "" H 8250 4850 30  0000 C CNN
-	1    8250 4850
-	0    1    1    0
-$EndComp
-Wire Wire Line
-	7300 4850 8100 4850
-Wire Wire Line
-	8400 4850 8600 4850
+P 8250 4950
+F 0 "R30" V 8330 4950 50  0000 C CNN
+F 1 "1k" V 8250 4950 50  0000 C CNN
+F 2 "" V 8180 4950 30  0000 C CNN
+F 3 "" H 8250 4950 30  0000 C CNN
+	1    8250 4950
+	0    1    1    0
+$EndComp
+Wire Wire Line
+	7300 4950 8100 4950
+Wire Wire Line
+	8400 4950 8600 4950
 $Comp
 L GND #PWR081
 U 1 1 5B178F7C
-P 9200 4850
-F 0 "#PWR081" H 9200 4600 50  0001 C CNN
-F 1 "GND" V 9200 4650 50  0000 C CNN
-F 2 "" H 9200 4850 60  0000 C CNN
-F 3 "" H 9200 4850 60  0000 C CNN
-	1    9200 4850
+P 9200 4950
+F 0 "#PWR081" H 9200 4700 50  0001 C CNN
+F 1 "GND" V 9200 4750 50  0000 C CNN
+F 2 "" H 9200 4950 60  0000 C CNN
+F 3 "" H 9200 4950 60  0000 C CNN
+	1    9200 4950
 	0    -1   -1   0
 $EndComp
 Wire Wire Line
-	9000 4850 9200 4850
+	9000 4950 9200 4950
+$Comp
+L PWR_FLAG #FLG082
+U 1 1 5B19051F
+P 8690 4230
+F 0 "#FLG082" H 8690 4325 50  0001 C CNN
+F 1 "PWR_FLAG" H 8690 4410 50  0000 C CNN
+F 2 "" H 8690 4230 50  0000 C CNN
+F 3 "" H 8690 4230 50  0000 C CNN
+	1    8690 4230
+	1    0    0    -1
+$EndComp
+Wire Wire Line
+	8690 4230 8690 4250
+Connection ~ 8690 4250
 $EndSCHEMATC

Commit message: finished drc
Parts:
- added R25: 50, symbol R
- renumbered R25 to R26, R26 to R27, R27 to R28, R28 to R29, R29 to R30, R30 to R31
Connections:
- net GND: now also U5.33, R25.2
- net MCLK4: now also R25.1
- no-connect marks 10 -> 8

Commit message: assign footprints
Parts:
- removed R25: 50, symbol R
- C42, C43, C46, C47, C48: footprint (none) -> fdsp_capacitor:C_1206_HandSoldering
- C44, C45, C49: footprint (none) -> fdsp_capacitor:C_Radial_D5_L11_P2
- D4, D5: footprint (none) -> fdsp_resistor:R_1206_HandSoldering
- R25: renamed from R26; footprint (none) -> fdsp_resistor:R_1206_HandSoldering
- R26: renamed from R27; footprint (none) -> fdsp_resistor:R_1206_HandSoldering
- R27: renamed from R28; footprint (none) -> fdsp_resistor:R_1206_HandSoldering
- R28: renamed from R29; footprint (none) -> fdsp_resistor:R_1206_HandSoldering
- R29: renamed from R30; footprint (none) -> fdsp_resistor:R_1206_HandSoldering
- R30: renamed from R31; footprint (none) -> fdsp_resistor:R_1206_HandSoldering
- U5: footprint CIR-QFN-32_5X5 -> footprints_CS8422-CNZ:CS8422-CNZ
Changed lines of the file:
@@
 F 0 "U5" H 5800 3550 60  0000 C CNN
 F 1 "CS8422-CNZ" H 5800 3450 60  0000 C CNN
-F 2 "CIR-QFN-32_5X5" H 5800 3390 60  0001 C CNN
+F 2 "footprints_CS8422-CNZ:CS8422-CNZ" H 5800 3390 60  0001 C CNN
 F 3 "" H 4300 3150 60  0000 C CNN
 	1    4300 3150
@@
 F 0 "C46" V 3350 3300 50  0000 L CNN
 F 1 "10n" V 3350 3050 50  0000 L CNN
-F 2 "" H 3438 3100 30  0000 C CNN
+F 2 "fdsp_capacitor:C_1206_HandSoldering" H 3438 3100 30  0001 C CNN
 F 3 "" H 3400 3250 60  0000 C CNN
 	1    3400 3250
@@
 F 0 "C43" H 2650 4500 50  0000 L CNN
 F 1 "100n" H 2550 4300 50  0000 L CNN
-F 2 "" H 2788 4250 30  0000 C CNN
+F 2 "fdsp_capacitor:C_1206_HandSoldering" H 2788 4250 30  0001 C CNN
 F 3 "" H 2750 4400 60  0000 C CNN
 	1    2750 4400
@@
 F 0 "C45" H 3075 4500 50  0000 L CNN
 F 1 "10µ" H 3075 4300 50  0000 L CNN
-F 2 "" H 3088 4250 30  0000 C CNN
+F 2 "fdsp_capacitor:C_Radial_D5_L11_P2" H 3088 4250 30  0001 C CNN
 F 3 "" H 3050 4400 60  0000 C CNN
 	1    3050 4400
@@
 F 0 "C48" H 8475 4500 50  0000 L CNN
 F 1 "100n" H 8475 4300 50  0000 L CNN
-F 2 "" H 8488 4250 30  0000 C CNN
+F 2 "fdsp_capacitor:C_1206_HandSoldering" H 8488 4250 30  0001 C CNN
 F 3 "" H 8450 4400 60  0000 C CNN
 	1    8450 4400
@@
 F 0 "C49" H 8775 4500 50  0000 L CNN
 F 1 "10µ" H 8775 4300 50  0000 L CNN
-F 2 "" H 8788 4250 30  0000 C CNN
+F 2 "fdsp_capacitor:C_Radial_D5_L11_P2" H 8788 4250 30  0001 C CNN
 F 3 "" H 8750 4400 60  0000 C CNN
 	1    8750 4400
@@
 F 0 "D4" H 8800 3450 50  0000 C CNN
 F 1 "LED" H 8800 3250 50  0000 C CNN
-F 2 "" H 8800 3350 60  0000 C CNN
+F 2 "fdsp_resistor:R_1206_HandSoldering" H 8800 3350 60  0001 C CNN
 F 3 "" H 8800 3350 60  0000 C CNN
 	1    8800 3350
@@
 $EndComp
 $Comp
-L R R30
+L R R29
 U 1 1 5B0AD1B9
 P 8250 3350
-F 0 "R30" V 8330 3350 50  0000 C CNN
+F 0 "R29" V 8330 3350 50  0000 C CNN
 F 1 "1k" V 8250 3350 50  0000 C CNN
-F 2 "" V 8180 3350 30  0000 C CNN
+F 2 "fdsp_resistor:R_1206_HandSoldering" V 8180 3350 30  0001 C CNN
 F 3 "" H 8250 3350 30  0000 C CNN
 	1    8250 3350
@@
 F 0 "C47" V 7900 4150 50  0000 L CNN
 F 1 "100n" V 7900 3800 50  0000 L CNN
-F 2 "" H 7988 3900 30  0000 C CNN
+F 2 "fdsp_capacitor:C_1206_HandSoldering" H 7988 3900 30  0001 C CNN
 F 3 "" H 7950 4050 60  0000 C CNN
 	1    7950 4050
@@
 NoConn ~ 7300 4550
 $Comp
-L R R28
+L R R27
 U 1 1 5B0AD987
 P 7700 4450
-F 0 "R28" V 7780 4450 50  0000 C CNN
+F 0 "R27" V 7780 4450 50  0000 C CNN
 F 1 "20k" V 7700 4450 50  0000 C CNN
-F 2 "" V 7630 4450 30  0000 C CNN
+F 2 "fdsp_resistor:R_1206_HandSoldering" V 7630 4450 30  0001 C CNN
 F 3 "" H 7700 4450 30  0000 C CNN
 	1    7700 4450
@@
 F 0 "C42" H 2650 3600 50  0000 L CNN
 F 1 "100n" H 2550 3400 50  0000 L CNN
-F 2 "" H 2788 3350 30  0000 C CNN
+F 2 "fdsp_capacitor:C_1206_HandSoldering" H 2788 3350 30  0001 C CNN
 F 3 "" H 2750 3500 60  0000 C CNN
 	1    2750 3500
@@
 F 0 "C44" H 3075 3600 50  0000 L CNN
 F 1 "10µ" H 3075 3400 50  0000 L CNN
-F 2 "" H 3088 3350 30  0000 C CNN
+F 2 "fdsp_capacitor:C_Radial_D5_L11_P2" H 3088 3350 30  0001 C CNN
 F 3 "" H 3050 3500 60  0000 C CNN
 	1    3050 3500
@@
 $EndComp
 $Comp
-L R R26
+L R R25
 U 1 1 5B0ADE1F
 P 3650 3750
-F 0 "R26" V 3730 3750 50  0000 C CNN
+F 0 "R25" V 3730 3750 50  0000 C CNN
 F 1 "32k4" V 3650 3750 50  0000 C CNN
-F 2 "" V 3580 3750 30  0000 C CNN
+F 2 "fdsp_resistor:R_1206_HandSoldering" V 3580 3750 30  0001 C CNN
 F 3 "" H 3650 3750 30  0000 C CNN
 	1    3650 3750
@@
 $EndComp
 $Comp
-L R R27
+L R R26
 U 1 1 5B0ADF07
 P 3650 3850
-F 0 "R27" V 3550 3850 50  0000 C CNN
+F 0 "R26" V 3550 3850 50  0000 C CNN
 F 1 "16k2" V 3650 3850 50  0000 C CNN
-F 2 "" V 3580 3850 30  0000 C CNN
+F 2 "fdsp_resistor:R_1206_HandSoldering" V 3580 3850 30  0001 C CNN
 F 3 "" H 3650 3850 30  0000 C CNN
 	1    3650 3850
@@
 $EndComp
 $Comp
-L R R29
+L R R28
 U 1 1 5B0AE799
 P 7700 4650
-F 0 "R29" V 7780 4650 50  0000 C CNN
+F 0 "R28" V 7780 4650 50  0000 C CNN
 F 1 "20k" V 7700 4650 50  0000 C CNN
-F 2 "" V 7630 4650 30  0000 C CNN
+F 2 "fdsp_resistor:R_1206_HandSoldering" V 7630 4650 30  0001 C CNN
 F 3 "" H 7700 4650 30  0000 C CNN
 	1    7700 4650
@@
 F 0 "D5" H 8800 5050 50  0000 C CNN
 F 1 "LED" H 8800 4850 50  0000 C CNN
-F 2 "" H 8800 4950 60  0000 C CNN
+F 2 "fdsp_resistor:R_1206_HandSoldering" H 8800 4950 60  0001 C CNN
 F 3 "" H 8800 4950 60  0000 C CNN
 	1    8800 4950
@@
 $EndComp
 $Comp
-L R R31
+L R R30
 U 1 1 5B178F74
 P 8250 4950
-F 0 "R31" V 8330 4950 50  0000 C CNN
+F 0 "R30" V 8330 4950 50  0000 C CNN
 F 1 "1k" V 8250 4950 50  0000 C CNN
-F 2 "" V 8180 4950 30  0000 C CNN
+F 2 "fdsp_resistor:R_1206_HandSoldering" V 8180 4950 30  0001 C CNN
 F 3 "" H 8250 4950 30  0000 C CNN
 	1    8250 4950
@@
 	1    0    0    -1
 $EndComp
-$Comp
-L R R25
-U 1 1 5B1F5FEA
-P 1990 4140
-F 0 "R25" V 2070 4140 50  0000 C CNN
-F 1 "50" V 1990 4140 50  0000 C CNN
-F 2 "" V 1920 4140 30  0000 C CNN
-F 3 "" H 1990 4140 30  0000 C CNN
-	1    1990 4140
-	1    0    0    -1
-$EndComp
 Wire Wire Line
 	4300 4350 4100 4350
@@
 Wire Wire Line
 	7620 3150 7620 3155
-Wire Wire Line
-	1990 3990 1990 3950
-Connection ~ 1990 3950
-$Comp
-L GND #PWR086
-U 1 1 5B1F6425
-P 1990 4340
-F 0 "#PWR086" H 1990 4090 50  0001 C CNN
-F 1 "GND" H 1990 4190 50  0000 C CNN
-F 2 "" H 1990 4340 60  0000 C CNN
-F 3 "" H 1990 4340 60  0000 C CNN
-	1    1990 4340
-	1    0    0    -1
-$EndComp
-Wire Wire Line
-	1990 4340 1990 4290
 $EndSCHEMATC

Commit message: almost done footprints
Parts:
- added P18: TST, fdsp_misc:Measurement_Point_Round-SMD-Pad_Small, symbol TST
Connections:
- net MCLK4: now also P18.1
Changed lines of the file:
@@
 Wire Wire Line
 	7620 3150 7620 3155
+$Comp
+L TST P18
+U 1 1 5B21909E
+P 1950 3900
+F 0 "P18" H 1950 4200 50  0000 C BNN
+F 1 "TST" H 1950 4150 50  0000 C CNN
+F 2 "fdsp_misc:Measurement_Point_Round-SMD-Pad_Small" H 1950 3900 50  0001 C CNN
+F 3 "" H 1950 3900 50  0000 C CNN
+	1    1950 3900
+	1    0    0    -1
+$EndComp
+Wire Wire Line
+	1950 3900 1950 3950
+Connection ~ 1950 3950
 $EndSCHEMATC

Commit message: kleine Anpassungen
Parts:
- R25: value 32k4 -> 32k4, 1%
- R26: value 16k2 -> 16k2, 1%
Connections:
- net +3V3: now also C47.2, U5.22 (VL)
Changed lines of the file:
@@
 P 3650 3750
 F 0 "R25" V 3730 3750 50  0000 C CNN
-F 1 "32k4" V 3650 3750 50  0000 C CNN
+F 1 "32k4, 1%" V 3650 3750 50  0000 C CNN
 F 2 "fdsp_resistor:R_1206_HandSoldering" V 3580 3750 30  0001 C CNN
 F 3 "" H 3650 3750 30  0000 C CNN
@@
 P 3650 3850
 F 0 "R26" V 3550 3850 50  0000 C CNN
-F 1 "16k2" V 3650 3850 50  0000 C CNN
+F 1 "16k2, 1%" V 3650 3850 50  0000 C CNN
 F 2 "fdsp_resistor:R_1206_HandSoldering" V 3580 3850 30  0001 C CNN
 F 3 "" H 3650 3850 30  0000 C CNN
@@
 	1950 3900 1950 3950
 Connection ~ 1950 3950
+$Comp
+L +3V3 #PWR?
+U 1 1 5B22C9D1
+P 7550 4050
+F 0 "#PWR?" H 7550 3900 50  0001 C CNN
+F 1 "+3V3" H 7550 4190 50  0000 C CNN
+F 2 "" H 7550 4050 60  0000 C CNN
+F 3 "" H 7550 4050 60  0000 C CNN
+	1    7550 4050
+	1    0    0    -1
+$EndComp
+Connection ~ 7550 4050
 $EndSCHEMATC
