File: SOURCES/power.sch (KiCad schematic (older format))
At the start: 19 parts, among them P13 CONN_01X02, U7 LM2842Y

Commit message: drc
Connections:
- net VIN: now also D7.2
Other:
- moved on the sheet: D7
Changed lines of the file:
@@
 L SMAJ28A D7
 U 1 1 5B11F195
-P 2940 3370
-F 0 "D7" H 2940 3370 60  0000 C CNN
-F 1 "SMAJ28A" H 2940 3110 60  0000 C CNN
-F 2 "" H 2940 3370 60  0001 C CNN
-F 3 "" H 2940 3370 60  0001 C CNN
-	1    2940 3370
+P 2940 3480
+F 0 "D7" H 2940 3480 60  0000 C CNN
+F 1 "SMAJ28A" H 2940 3220 60  0000 C CNN
+F 2 "" H 2940 3480 60  0001 C CNN
+F 3 "" H 2940 3480 60  0001 C CNN
+	1    2940 3480
 	0    1    1    0
 $EndComp
@@
 	1080 3830 9270 3830
 Wire Wire Line
-	2810 3650 2810 3830
+	2810 3760 2810 3830
 Connection ~ 2810 3830
 Wire Wire Line
@@
 	1    0    0    -1
 $EndComp
+Wire Wire Line
+	2810 3190 2810 3070
+Connection ~ 2810 3070
 $EndSCHEMATC

Commit message: finished drc
Parts:
- renumbered R35 to R37, R36 to R38
Changed lines of the file:
@@
 $EndComp
 $Comp
-L R R35
+L R R37
 U 1 1 5B12302F
 P 7040 3610
-F 0 "R35" V 7120 3610 50  0000 C CNN
+F 0 "R37" V 7120 3610 50  0000 C CNN
 F 1 "1.02k" V 7040 3610 50  0000 C CNN
 F 2 "" V 6970 3610 30  0000 C CNN
@@
 $EndComp
 $Comp
-L R R36
+L R R38
 U 1 1 5B123449
 P 8060 3370
-F 0 "R36" V 8140 3370 50  0000 C CNN
+F 0 "R38" V 8140 3370 50  0000 C CNN
 F 1 "3.4k" V 8060 3370 50  0000 C CNN
 F 2 "" V 7990 3370 30  0000 C CNN
@@
 $EndComp
 $Comp
-L +3V3 #PWR097
+L +3V3 #PWR0105
 U 1 1 5B12407E
 P 8930 3030
-F 0 "#PWR097" H 8930 2880 50  0001 C CNN
+F 0 "#PWR0105" H 8930 2880 50  0001 C CNN
 F 1 "+3V3" H 8930 3170 50  0000 C CNN
 F 2 "" H 8930 3030 60  0000 C CNN
@@
 Connection ~ 8930 3830
 $Comp
-L GND #PWR098
+L GND #PWR0106
 U 1 1 5B1264D3
 P 7480 3970
-F 0 "#PWR098" H 7480 3720 50  0001 C CNN
+F 0 "#PWR0106" H 7480 3720 50  0001 C CNN
 F 1 "GND" H 7480 3820 50  0000 C CNN
 F 2 "" H 7480 3970 60  0000 C CNN
@@
 Connection ~ 7040 3830
 $Comp
-L VCC #PWR099
+L VCC #PWR0107
 U 1 1 5B1283A5
 P 4900 3010
-F 0 "#PWR099" H 4900 2860 50  0001 C CNN
+F 0 "#PWR0107" H 4900 2860 50  0001 C CNN
 F 1 "VCC" H 4900 3160 50  0000 C CNN
 F 2 "" H 4900 3010 60  0000 C CNN
@@
 $EndComp
 $Comp
-L PWR_FLAG #FLG0100
+L PWR_FLAG #FLG0108
 U 1 1 5B12846A
 P 5250 3020
-F 0 "#FLG0100" H 5250 3115 50  0001 C CNN
+F 0 "#FLG0108" H 5250 3115 50  0001 C CNN
 F 1 "PWR_FLAG" H 5250 3200 50  0000 C CNN
 F 2 "" H 5250 3020 50  0000 C CNN
@@
 $EndComp
 $Comp
-L +12V #PWR0101
+L +12V #PWR0109
 U 1 1 5B12FB51
 P 1030 3040
-F 0 "#PWR0101" H 1030 2890 50  0001 C CNN
+F 0 "#PWR0109" H 1030 2890 50  0001 C CNN
 F 1 "+12V" H 1030 3180 50  0000 C CNN
 F 2 "" H 1030 3040 60  0000 C CNN
@@
 $EndComp
 $Comp
-L PWR_FLAG #FLG0102
+L PWR_FLAG #FLG0110
 U 1 1 5B12FD62
 P 1210 2940
-F 0 "#FLG0102" H 1210 3035 50  0001 C CNN
+F 0 "#FLG0110" H 1210 3035 50  0001 C CNN
 F 1 "PWR_FLAG" H 1210 3120 50  0000 C CNN
 F 2 "" H 1210 2940 50  0000 C CNN
@@
 	1600 3070 1690 3070
 $Comp
-L VIN #PWR0103
+L VIN #PWR0111
 U 1 1 5B130AA6
 P 3620 3010
-F 0 "#PWR0103" H 3620 2860 50  0001 C CNN
+F 0 "#PWR0111" H 3620 2860 50  0001 C CNN
 F 1 "VIN" H 3620 3150 50  0000 C CNN
 F 2 "" H 3620 3010 60  0000 C CNN
@@
 $EndComp
 $Comp
-L PWR_FLAG #FLG0104
+L PWR_FLAG #FLG0112
 U 1 1 5B130AE0
 P 3300 2990
-F 0 "#FLG0104" H 3300 3085 50  0001 C CNN
+F 0 "#FLG0112" H 3300 3085 50  0001 C CNN
 F 1 "PWR_FLAG" H 3300 3170 50  0000 C CNN
 F 2 "" H 3300 2990 50  0000 C CNN

Commit message: assign footprints
Parts:
- added D10: LED, fdsp_resistor:R_1206_HandSoldering, symbol LED
- added R46: 330, fdsp_resistor:R_1206_HandSoldering, symbol R
- C60, C61, C63, C64, C65, C66, C67, C68: footprint (none) -> fdsp_capacitor:C_1206_HandSoldering
- C62: footprint (none) -> fdsp_capacitor:C_Radial_D5_L11_P2
- D6, D7, D8: footprint (none) -> fdsp_diode:SMA
- F1: footprint (none) -> fdsp_resistor:R_1206_HandSoldering
- FB2: value BLM18PG471SNL -> BLM18PG471SN1; footprint (none) -> fdsp_resistor:R_0603_HandSoldering
- P13: footprint (none) -> fdsp_connector:RIACON101-2
- R35: renamed from R37; footprint (none) -> fdsp_resistor:R_1206_HandSoldering
- R36: renamed from R38; footprint (none) -> fdsp_resistor:R_1206_HandSoldering
Connections:
- net +3V3: now also R46.1
- net GND: now also D10.1 (K)
- new net: D10.2 (A), R46.2
Changed lines of the file:
@@
 F 0 "U7" H 6530 3520 60  0000 C CNN
 F 1 "LM2842Y" H 6180 3520 60  0000 C CNN
-F 2 "" H 6330 3220 60  0000 C CNN
+F 2 "" H 6330 3220 60  0001 C CNN
 F 3 "" H 6330 3220 60  0000 C CNN
 	1    6280 3220
@@
 F 0 "P13" H 790 3270 50  0000 C CNN
 F 1 "CONN_01X02" V 890 3120 50  0000 C CNN
-F 2 "" H 790 3120 60  0000 C CNN
+F 2 "fdsp_connector:RIACON101-2" H 790 3120 60  0001 C CNN
 F 3 "" H 790 3120 60  0000 C CNN
 	1    790  3120
@@
 F 0 "D6" H 1450 3170 50  0000 C CNN
 F 1 "D_Schottky" H 1450 2970 50  0000 C CNN
-F 2 "" H 1450 3070 60  0000 C CNN
+F 2 "fdsp_diode:SMA" H 1450 3070 60  0001 C CNN
 F 3 "" H 1450 3070 60  0000 C CNN
 	1    1450 3070
@@
 F 0 "F1" H 2160 2700 60  0000 C CNN
 F 1 "0ZCJ0050AF2E" H 2140 2940 60  0000 C CNN
-F 2 "" H 2140 2940 60  0001 C CNN
+F 2 "fdsp_resistor:R_1206_HandSoldering" H 2140 2940 60  0001 C CNN
 F 3 "" H 2140 2940 60  0001 C CNN
 	1    2390 2940
@@
 F 0 "D7" H 2940 3480 60  0000 C CNN
 F 1 "SMAJ28A" H 2940 3220 60  0000 C CNN
-F 2 "" H 2940 3480 60  0001 C CNN
+F 2 "fdsp_diode:SMA" H 2940 3480 60  0001 C CNN
 F 3 "" H 2940 3480 60  0001 C CNN
 	1    2940 3480
@@
 F 0 "C60" H 3325 3450 50  0000 L CNN
 F 1 "100n" H 3325 3250 50  0000 L CNN
-F 2 "" H 3338 3200 30  0000 C CNN
+F 2 "fdsp_capacitor:C_1206_HandSoldering" H 3338 3200 30  0001 C CNN
 F 3 "" H 3300 3350 60  0000 C CNN
 	1    3300 3350
@@
 F 0 "C61" H 3645 3450 50  0000 L CNN
 F 1 "10u" H 3645 3250 50  0000 L CNN
-F 2 "" H 3658 3200 30  0000 C CNN
+F 2 "fdsp_capacitor:C_1206_HandSoldering" H 3658 3200 30  0001 C CNN
 F 3 "" H 3620 3350 60  0000 C CNN
 	1    3620 3350
@@
 P 4240 3070
 F 0 "FB2" H 4240 3220 50  0000 C CNN
-F 1 "BLM18PG471SNL" H 4240 2970 50  0000 C CNN
-F 2 "" H 4240 3070 50  0000 C CNN
+F 1 "BLM18PG471SN1" H 4240 2970 50  0000 C CNN
+F 2 "fdsp_resistor:R_0603_HandSoldering" H 4240 3070 50  0001 C CNN
 F 3 "" H 4240 3070 50  0000 C CNN
 	1    4240 3070
@@
 F 0 "C62" H 4925 3440 50  0000 L CNN
 F 1 "100u" H 4925 3240 50  0000 L CNN
-F 2 "" H 4938 3190 30  0000 C CNN
+F 2 "fdsp_capacitor:C_Radial_D5_L11_P2" H 4938 3190 30  0001 C CNN
 F 3 "" H 4900 3340 60  0000 C CNN
 	1    4900 3340
@@
 F 0 "C63" H 5275 3450 50  0000 L CNN
 F 1 "10u" H 5275 3250 50  0000 L CNN
-F 2 "" H 5288 3200 30  0000 C CNN
+F 2 "fdsp_capacitor:C_1206_HandSoldering" H 5288 3200 30  0001 C CNN
 F 3 "" H 5250 3350 60  0000 C CNN
 	1    5250 3350
@@
 F 0 "C64" H 5545 3450 50  0000 L CNN
 F 1 "100n" H 5545 3250 50  0000 L CNN
-F 2 "" H 5558 3200 30  0000 C CNN
+F 2 "fdsp_capacitor:C_1206_HandSoldering" H 5558 3200 30  0001 C CNN
 F 3 "" H 5520 3350 60  0000 C CNN
 	1    5520 3350
@@
 F 0 "C65" H 7185 3170 50  0000 L CNN
 F 1 "150n" H 6940 2970 50  0000 L CNN
-F 2 "" H 7198 2920 30  0000 C CNN
+F 2 "fdsp_capacitor:C_1206_HandSoldering" H 7198 2920 30  0001 C CNN
 F 3 "" H 7160 3070 60  0000 C CNN
 	1    7160 3070
@@
 $EndComp
 $Comp
-L R R37
+L R R35
 U 1 1 5B12302F
 P 7040 3610
-F 0 "R37" V 7120 3610 50  0000 C CNN
+F 0 "R35" V 7120 3610 50  0000 C CNN
 F 1 "1.02k" V 7040 3610 50  0000 C CNN
-F 2 "" V 6970 3610 30  0000 C CNN
+F 2 "fdsp_resistor:R_1206_HandSoldering" V 6970 3610 30  0001 C CNN
 F 3 "" H 7040 3610 30  0000 C CNN
 	1    7040 3610
@@
 F 0 "D8" H 7480 3710 50  0000 C CNN
 F 1 "B150" H 7480 3510 50  0000 C CNN
-F 2 "" H 7480 3610 60  0000 C CNN
+F 2 "fdsp_diode:SMA" H 7480 3610 60  0001 C CNN
 F 3 "" H 7480 3610 60  0000 C CNN
 	1    7480 3610
@@
 F 0 "L5" H 8050 3170 50  0000 C CNN
 F 1 "47u" H 8050 3020 50  0000 C CNN
-F 2 "" H 8050 3070 50  0000 C CNN
+F 2 "" H 8050 3070 50  0001 C CNN
 F 3 "" H 8050 3070 50  0000 C CNN
 	1    8050 3070
@@
 $EndComp
 $Comp
-L R R38
+L R R36
 U 1 1 5B123449
 P 8060 3370
-F 0 "R38" V 8140 3370 50  0000 C CNN
+F 0 "R36" V 8140 3370 50  0000 C CNN
 F 1 "3.4k" V 8060 3370 50  0000 C CNN
-F 2 "" V 7990 3370 30  0000 C CNN
+F 2 "fdsp_resistor:R_1206_HandSoldering" V 7990 3370 30  0001 C CNN
 F 3 "" H 8060 3370 30  0000 C CNN
 	1    8060 3370
@@
 F 0 "C66" H 8645 3420 50  0000 L CNN
 F 1 "100n" H 8645 3220 50  0000 L CNN
-F 2 "" H 8658 3170 30  0000 C CNN
+F 2 "fdsp_capacitor:C_1206_HandSoldering" H 8658 3170 30  0001 C CNN
 F 3 "" H 8620 3320 60  0000 C CNN
 	1    8620 3320
@@
 F 0 "C67" H 8955 3420 50  0000 L CNN
 F 1 "10u" H 8955 3220 50  0000 L CNN
-F 2 "" H 8968 3170 30  0000 C CNN
+F 2 "fdsp_capacitor:C_1206_HandSoldering" H 8968 3170 30  0001 C CNN
 F 3 "" H 8930 3320 60  0000 C CNN
 	1    8930 3320
@@
 F 0 "C68" H 9295 3420 50  0000 L CNN
 F 1 "10u" H 9295 3220 50  0000 L CNN
-F 2 "" H 9308 3170 30  0000 C CNN
+F 2 "fdsp_capacitor:C_1206_HandSoldering" H 9308 3170 30  0001 C CNN
 F 3 "" H 9270 3320 60  0000 C CNN
 	1    9270 3320
@@
 $EndComp
 $Comp
-L +3V3 #PWR0105
+L +3V3 #PWR0103
 U 1 1 5B12407E
 P 8930 3030
-F 0 "#PWR0105" H 8930 2880 50  0001 C CNN
+F 0 "#PWR0103" H 8930 2880 50  0001 C CNN
 F 1 "+3V3" H 8930 3170 50  0000 C CNN
 F 2 "" H 8930 3030 60  0000 C CNN
@@
 	1080 3170 1080 3830
 Wire Wire Line
-	1080 3830 9270 3830
+	1080 3830 9635 3830
 Wire Wire Line
 	2810 3760 2810 3830
@@
 Connection ~ 7040 3370
 Wire Wire Line
-	8300 3070 9270 3070
+	8300 3070 9635 3070
 Wire Wire Line
 	8210 3370 8350 3370
@@
 Connection ~ 8930 3830
 $Comp
-L GND #PWR0106
+L GND #PWR0104
 U 1 1 5B1264D3
 P 7480 3970
-F 0 "#PWR0106" H 7480 3720 50  0001 C CNN
+F 0 "#PWR0104" H 7480 3720 50  0001 C CNN
 F 1 "GND" H 7480 3820 50  0000 C CNN
 F 2 "" H 7480 3970 60  0000 C CNN
@@
 Connection ~ 7040 3830
 $Comp
-L VCC #PWR0107
+L VCC #PWR0105
 U 1 1 5B1283A5
 P 4900 3010
-F 0 "#PWR0107" H 4900 2860 50  0001 C CNN
+F 0 "#PWR0105" H 4900 2860 50  0001 C CNN
 F 1 "VCC" H 4900 3160 50  0000 C CNN
 F 2 "" H 4900 3010 60  0000 C CNN
@@
 $EndComp
 $Comp
-L PWR_FLAG #FLG0108
+L PWR_FLAG #FLG0106
 U 1 1 5B12846A
 P 5250 3020
-F 0 "#FLG0108" H 5250 3115 50  0001 C CNN
+F 0 "#FLG0106" H 5250 3115 50  0001 C CNN
 F 1 "PWR_FLAG" H 5250 3200 50  0000 C CNN
 F 2 "" H 5250 3020 50  0000 C CNN
@@
 $EndComp
 $Comp
-L +12V #PWR0109
+L +12V #PWR0107
 U 1 1 5B12FB51
 P 1030 3040
-F 0 "#PWR0109" H 1030 2890 50  0001 C CNN
+F 0 "#PWR0107" H 1030 2890 50  0001 C CNN
 F 1 "+12V" H 1030 3180 50  0000 C CNN
 F 2 "" H 1030 3040 60  0000 C CNN
@@
 $EndComp
 $Comp
-L PWR_FLAG #FLG0110
+L PWR_FLAG #FLG0108
 U 1 1 5B12FD62
 P 1210 2940
-F 0 "#FLG0110" H 1210 3035 50  0001 C CNN
+F 0 "#FLG0108" H 1210 3035 50  0001 C CNN
 F 1 "PWR_FLAG" H 1210 3120 50  0000 C CNN
 F 2 "" H 1210 2940 50  0000 C CNN
@@
 	1600 3070 1690 3070
 $Comp
-L VIN #PWR0111
+L VIN #PWR0109
 U 1 1 5B130AA6
 P 3620 3010
-F 0 "#PWR0111" H 3620 2860 50  0001 C CNN
+F 0 "#PWR0109" H 3620 2860 50  0001 C CNN
 F 1 "VIN" H 3620 3150 50  0000 C CNN
 F 2 "" H 3620 3010 60  0000 C CNN
@@
 $EndComp
 $Comp
-L PWR_FLAG #FLG0112
+L PWR_FLAG #FLG0110
 U 1 1 5B130AE0
 P 3300 2990
-F 0 "#FLG0112" H 3300 3085 50  0001 C CNN
+F 0 "#FLG0110" H 3300 3085 50  0001 C CNN
 F 1 "PWR_FLAG" H 3300 3170 50  0000 C CNN
 F 2 "" H 3300 2990 50  0000 C CNN
@@
 	2810 3190 2810 3070
 Connection ~ 2810 3070
+$Comp
+L LED D10
+U 1 1 5B207F31
+P 9635 3620
+F 0 "D10" H 9635 3720 50  0000 C CNN
+F 1 "LED" H 9635 3520 50  0000 C CNN
+F 2 "fdsp_resistor:R_1206_HandSoldering" H 9635 3620 60  0001 C CNN
+F 3 "" H 9635 3620 60  0000 C CNN
+	1    9635 3620
+	0    -1   -1   0
+$EndComp
+$Comp
+L R R46
+U 1 1 5B2080CB
+P 9635 3235
+F 0 "R46" V 9715 3235 50  0000 C CNN
+F 1 "330" V 9635 3235 50  0000 C CNN
+F 2 "fdsp_resistor:R_1206_HandSoldering" V 9565 3235 30  0001 C CNN
+F 3 "" H 9635 3235 30  0000 C CNN
+	1    9635 3235
+	1    0    0    -1
+$EndComp
+Wire Wire Line
+	9635 3070 9635 3085
+Connection ~ 9270 3070
+Wire Wire Line
+	9635 3830 9635 3820
+Connection ~ 9270 3830
+Wire Wire Line
+	9635 3385 9635 3420
 $EndSCHEMATC

Commit message: almost done footprints
Parts:
- L5: footprint (none) -> fdsp_inductor:Choke_SMD_6.0x5.8
- U7: footprint (none) -> fdsp_housing:SOT23-6_1.7x3.0mm_Pitch0.95mm
Changed lines of the file:
@@
 F 0 "U7" H 6530 3520 60  0000 C CNN
 F 1 "LM2842Y" H 6180 3520 60  0000 C CNN
-F 2 "" H 6330 3220 60  0001 C CNN
+F 2 "fdsp_housing:SOT23-6_1.7x3.0mm_Pitch0.95mm" H 6330 3220 60  0001 C CNN
 F 3 "" H 6330 3220 60  0000 C CNN
 	1    6280 3220
@@
 F 0 "L5" H 8050 3170 50  0000 C CNN
 F 1 "47u" H 8050 3020 50  0000 C CNN
-F 2 "" H 8050 3070 50  0001 C CNN
+F 2 "fdsp_inductor:Choke_SMD_6.0x5.8" H 8050 3070 50  0001 C CNN
 F 3 "" H 8050 3070 50  0000 C CNN
 	1    8050 3070

Commit message: almost done footprints
Parts:
- added P20: TST, fdsp_misc:Measurement_Point_Round-SMD-Pad_Small, symbol TST
Connections:
- net +3V3: now also P20.1
Changed lines of the file:
@@
 Connection ~ 8930 3070
 Wire Wire Line
-	9270 3070 9270 3170
+	9270 2980 9270 3170
 Wire Wire Line
 	9270 3830 9270 3470
@@
 Wire Wire Line
 	9635 3385 9635 3420
+$Comp
+L TST P20
+U 1 1 5B2196E9
+P 9270 2980
+F 0 "P20" H 9270 3280 50  0000 C BNN
+F 1 "TST" H 9270 3230 50  0000 C CNN
+F 2 "fdsp_misc:Measurement_Point_Round-SMD-Pad_Small" H 9270 2980 50  0001 C CNN
+F 3 "" H 9270 2980 50  0000 C CNN
+	1    9270 2980
+	1    0    0    -1
+$EndComp
 $EndSCHEMATC
