File: SOURCES/power.sch (KiCad schematic (older format))
At the start: 22 parts, among them P13 CONN_01X02, P20 TST, U7 LM2842Y

Commit message: Bauteilliste
Parts:
- D10: value LED -> LED_GREEN
Changed lines of the file:
@@
 $EndComp
 $Comp
-L +3V3 #PWR0103
+L +3V3 #PWR0104
 U 1 1 5B12407E
 P 8930 3030
-F 0 "#PWR0103" H 8930 2880 50  0001 C CNN
+F 0 "#PWR0104" H 8930 2880 50  0001 C CNN
 F 1 "+3V3" H 8930 3170 50  0000 C CNN
 F 2 "" H 8930 3030 60  0000 C CNN
@@
 Connection ~ 8930 3830
 $Comp
-L GND #PWR0104
+L GND #PWR0105
 U 1 1 5B1264D3
 P 7480 3970
-F 0 "#PWR0104" H 7480 3720 50  0001 C CNN
+F 0 "#PWR0105" H 7480 3720 50  0001 C CNN
 F 1 "GND" H 7480 3820 50  0000 C CNN
 F 2 "" H 7480 3970 60  0000 C CNN
@@
 Connection ~ 7040 3830
 $Comp
-L VCC #PWR0105
+L VCC #PWR0106
 U 1 1 5B1283A5
 P 4900 3010
-F 0 "#PWR0105" H 4900 2860 50  0001 C CNN
+F 0 "#PWR0106" H 4900 2860 50  0001 C CNN
 F 1 "VCC" H 4900 3160 50  0000 C CNN
 F 2 "" H 4900 3010 60  0000 C CNN
@@
 $EndComp
 $Comp
-L PWR_FLAG #FLG0106
+L PWR_FLAG #FLG0107
 U 1 1 5B12846A
 P 5250 3020
-F 0 "#FLG0106" H 5250 3115 50  0001 C CNN
+F 0 "#FLG0107" H 5250 3115 50  0001 C CNN
 F 1 "PWR_FLAG" H 5250 3200 50  0000 C CNN
 F 2 "" H 5250 3020 50  0000 C CNN
@@
 $EndComp
 $Comp
-L +12V #PWR0107
+L +12V #PWR0108
 U 1 1 5B12FB51
 P 1030 3040
-F 0 "#PWR0107" H 1030 2890 50  0001 C CNN
+F 0 "#PWR0108" H 1030 2890 50  0001 C CNN
 F 1 "+12V" H 1030 3180 50  0000 C CNN
 F 2 "" H 1030 3040 60  0000 C CNN
@@
 $EndComp
 $Comp
-L PWR_FLAG #FLG0108
+L PWR_FLAG #FLG0109
 U 1 1 5B12FD62
 P 1210 2940
-F 0 "#FLG0108" H 1210 3035 50  0001 C CNN
+F 0 "#FLG0109" H 1210 3035 50  0001 C CNN
 F 1 "PWR_FLAG" H 1210 3120 50  0000 C CNN
 F 2 "" H 1210 2940 50  0000 C CNN
@@
 	1600 3070 1690 3070
 $Comp
-L VIN #PWR0109
+L VIN #PWR0110
 U 1 1 5B130AA6
 P 3620 3010
-F 0 "#PWR0109" H 3620 2860 50  0001 C CNN
+F 0 "#PWR0110" H 3620 2860 50  0001 C CNN
 F 1 "VIN" H 3620 3150 50  0000 C CNN
 F 2 "" H 3620 3010 60  0000 C CNN
@@
 $EndComp
 $Comp
-L PWR_FLAG #FLG0110
+L PWR_FLAG #FLG0111
 U 1 1 5B130AE0
 P 3300 2990
-F 0 "#FLG0110" H 3300 3085 50  0001 C CNN
+F 0 "#FLG0111" H 3300 3085 50  0001 C CNN
 F 1 "PWR_FLAG" H 3300 3170 50  0000 C CNN
 F 2 "" H 3300 2990 50  0000 C CNN
@@
 P 9635 3620
 F 0 "D10" H 9635 3720 50  0000 C CNN
-F 1 "LED" H 9635 3520 50  0000 C CNN
+F 1 "LED_GREEN" H 9635 3520 50  0000 C CNN
 F 2 "fdsp_resistor:R_1206_HandSoldering" H 9635 3620 60  0001 C CNN
 F 3 "" H 9635 3620 60  0000 C CNN

Commit message: layout
Parts:
- C62: footprint fdsp_capacitor:C_Radial_D5_L11_P2 -> fdsp_capacitor:C_Radial_D6.3_L11.2_P2.5
Changed lines of the file:
@@
 F 0 "C62" H 4925 3440 50  0000 L CNN
 F 1 "100u" H 4925 3240 50  0000 L CNN
-F 2 "fdsp_capacitor:C_Radial_D5_L11_P2" H 4938 3190 30  0001 C CNN
+F 2 "fdsp_capacitor:C_Radial_D6.3_L11.2_P2.5" H 4938 3190 30  0001 C CNN
 F 3 "" H 4900 3340 60  0000 C CNN
 	1    4900 3340

Commit message: added choke footprint
Parts:
- L5: footprint fdsp_inductor:Choke_SMD_6.0x5.8 -> Choke_SMD_10:Choke_SMD_10.1x10.0
Changed lines of the file:
@@
 F 0 "L5" H 8050 3170 50  0000 C CNN
 F 1 "47u" H 8050 3020 50  0000 C CNN
-F 2 "fdsp_inductor:Choke_SMD_6.0x5.8" H 8050 3070 50  0001 C CNN
+F 2 "Choke_SMD_10:Choke_SMD_10.1x10.0" H 8050 3070 50  0001 C CNN
 F 3 "" H 8050 3070 50  0000 C CNN
 	1    8050 3070

Commit message: updated references
Parts:
- R35: value 1.02k -> 1k02
- R36: value 3.4k -> 3k4
Changed lines of the file:
@@
 P 7040 3610
 F 0 "R35" V 7120 3610 50  0000 C CNN
-F 1 "1.02k" V 7040 3610 50  0000 C CNN
+F 1 "1k02" V 7040 3610 50  0000 C CNN
 F 2 "fdsp_resistor:R_1206_HandSoldering" V 6970 3610 30  0001 C CNN
 F 3 "" H 7040 3610 30  0000 C CNN
@@
 P 8060 3370
 F 0 "R36" V 8140 3370 50  0000 C CNN
-F 1 "3.4k" V 8060 3370 50  0000 C CNN
+F 1 "3k4" V 8060 3370 50  0000 C CNN
 F 2 "fdsp_resistor:R_1206_HandSoldering" V 7990 3370 30  0001 C CNN
 F 3 "" H 8060 3370 30  0000 C CNN
