File: SOURCES/smd_aio.sch (KiCad schematic (older format))
At the start: 62 parts, among them J1 RCA_01, J2 RCA_01, P1 CONN_01X06, P2 CONN_01X03, P3 CONN_02X05, P4 STDCONN, P5 CONN_01X04, P6 CONN_02X04, P7 CONN_02X04, Q1 BSS123, Q2 BSS123, Q3 BSS123, Q4 BSS123, Q5 FZT751TA, SW1 SW_PUSH, U1 ADAU1701, U2 24AA256SN

Commit message: design rule check
Parts:
- gave numbers to parts that had none: 1
- renumbered P2 to P3, P3 to P4, P4 to P5, P5 to P6, P6 to P7, P7 to P8
Connections:
- net MP4: now reaches U1.8 (MP4)
- net MP5: now reaches U1.9 (MP5)

Commit message: design rule check
Connections:
- net +3V3: now also C5.1, C6.2, Q5.3 (E), U1.18 (IOVDD)
- net +5V: now also Q1.1 (G)
- net GND: now also U1.12 (DGND)
- net at U1.13 (DVDD), U1.24 (DVDD): now also C3.1, C4.1
Changed lines of the file:
@@
 LIBS:fdsp_transistor_new
 LIBS:LM2738XMY&slash_NOPB-symbols
+LIBS:smd_aio-cache
 EELAYER 25 0
 EELAYER END
@@
 $EndComp
 Wire Wire Line
-	4010 4540 4010 4465
-Wire Wire Line
 	3370 4540 4380 4540
 Wire Wire Line
@@
 Connection ~ 3840 1860
 Wire Wire Line
-	4410 1200 4410 1940
+	4410 1100 4410 1940
 Wire Wire Line
 	4410 1570 4420 1570
@@
 Wire Wire Line
 	4720 1300 4720 1750
-Wire Wire Line
-	4080 1010 4080 1550
-Wire Wire Line
-	4040 1200 4410 1200
 Wire Wire Line
 	4410 1940 3920 1940
@@
 Wire Wire Line
 	2430 5770 2430 6130
-Wire Wire Line
-	1990 6240 1990 5960
-Wire Wire Line
-	1990 5960 2430 5960
 Connection ~ 2430 5960
 Wire Wire Line
@@
 Wire Wire Line
 	2720 2310 2650 2310
+Wire Wire Line
+	1990 6210 1990 5960
+Wire Wire Line
+	1990 5960 2430 5960
+Wire Wire Line
+	4010 4470 4010 4540
+Wire Wire Line
+	3390 1470 3520 1470
+Connection ~ 3520 1470
+Wire Wire Line
+	3390 1760 3520 1760
+Connection ~ 3520 1760
+Wire Wire Line
+	4080 1010 4080 1550
+Wire Wire Line
+	4040 1200 4080 1200
+Connection ~ 4080 1200
+Wire Wire Line
+	4080 1100 4410 1100
+Connection ~ 4080 1100
 $EndSCHEMATC

Commit message: finished drc
Parts:
- removed P2: CONN_01X02, symbol CONN_01X02
- added P2: CONN_01X04, symbol CONN_01X04
Connections:
- net +3V3: now also P2.1 (P1)
- net GND: now also P2.2 (P2)
- net MP2: now also P2.3 (P3)
- net MP3: now also P2.4 (P4)
Other:
- note added: "MPs_IN & 3v3;GND"
- note removed: "MPs_IN"
Changed lines of the file:
@@
 Text Notes 10280 5990 0    76   ~ 15
 Input
-$Comp
-L CONN_01X02 P2
-U 1 1 5B102BB9
-P 4180 8790
-F 0 "P2" H 4180 8940 50  0000 C CNN
-F 1 "CONN_01X02" V 4280 8790 50  0000 C CNN
-F 2 "" H 4180 8790 60  0000 C CNN
-F 3 "" H 4180 8790 60  0000 C CNN
-	1    4180 8790
-	1    0    0    -1
-$EndComp
 Text GLabel 3980 8740 0    52   BiDi ~ 0
 MP2
 Text GLabel 3980 8840 0    52   BiDi ~ 0
 MP3
-Text Notes 3810 8480 0    76   ~ 15
-MPs_IN
+Text Notes 3515 8255 0    76   ~ 15
+MPs_IN & 3v3;GND
 Text GLabel 2650 2710 0    52   Input ~ 0
 MP4
@@
 	4080 1100 4410 1100
 Connection ~ 4080 1100
+$Comp
+L CONN_01X04 P2
+U 1 1 5B1EB9BC
+P 4180 8690
+F 0 "P2" H 4180 8940 50  0000 C CNN
+F 1 "CONN_01X04" V 4280 8690 50  0000 C CNN
+F 2 "" H 4180 8690 60  0000 C CNN
+F 3 "" H 4180 8690 60  0000 C CNN
+	1    4180 8690
+	1    0    0    -1
+$EndComp
+$Comp
+L +3V3 #PWR039
+U 1 1 5B1ED1B0
+P 3980 8540
+F 0 "#PWR039" H 3980 8390 50  0001 C CNN
+F 1 "+3V3" H 3980 8680 50  0000 C CNN
+F 2 "" H 3980 8540 60  0000 C CNN
+F 3 "" H 3980 8540 60  0000 C CNN
+	1    3980 8540
+	1    0    0    -1
+$EndComp
+$Comp
+L GND #PWR040
+U 1 1 5B1ED240
+P 3645 8655
+F 0 "#PWR040" H 3645 8405 50  0001 C CNN
+F 1 "GND" H 3645 8505 50  0000 C CNN
+F 2 "" H 3645 8655 60  0000 C CNN
+F 3 "" H 3645 8655 60  0000 C CNN
+	1    3645 8655
+	1    0    0    -1
+$EndComp
+Wire Wire Line
+	3645 8655 3645 8640
+Wire Wire Line
+	3645 8640 3980 8640
 $EndSCHEMATC

Commit message: assign footprints
Parts:
- C10, C11, C12, C14, C15, C16, C17, C18, C19, C3, C4, C6, C8, C9: footprint (none) -> fdsp_capacitor:C_1206_HandSoldering
- C13, C2, C5, C7: footprint (none) -> fdsp_capacitor:C_Radial_D5_L11_P2
- D1, D2: footprint (none) -> fdsp_diode:SMA
- P2: footprint (none) -> fdsp_pinheader:Pin_Header_Straight_1x04
- P3: footprint (none) -> fdsp_pinheader:Pin_Header_Straight_1x03
- P4: footprint (none) -> fdsp_connector:IDC_Header_Straight_10pins
- P6: footprint fdsp_pinheader:Pin_Header_Angled_1x04 -> fdsp_pinheader:Pin_Header_Straight_1x04
- Q1, Q2, Q3, Q4: footprint (none) -> fdsp_housing_new:SOT-23_Handsoldering
- Q5: footprint (none) -> fdsp_housing_new:SOT-223
- R1, R10, R11, R2, R3, R4, R5, R6, R7, R8, R9: footprint (none) -> fdsp_resistor:R_1206_HandSoldering
- SW1: footprint (none) -> fdsp_housing_new:SW_PUSH_6mm
- U1: footprint TQFP48 -> fdsp_housing_new:LQFP-48_7x7mm_Pitch0.5mm
- U2: footprint (none) -> fdsp_housing_new:SOIC-8_3.9x4.9mm_Pitch1.27mm

Commit message: almost done footprints
Parts:
- added P16: TST, fdsp_misc:Measurement_Point_Round-SMD-Pad_Small, symbol TST
Connections:
- net MCLK0: now also P16.1
Changed lines of the file:
@@
 Wire Wire Line
 	3645 8640 3980 8640
+$Comp
+L TST P16
+U 1 1 5B217DC8
+P 5250 2525
+F 0 "P16" H 5250 2825 50  0000 C BNN
+F 1 "TST" H 5250 2775 50  0000 C CNN
+F 2 "fdsp_misc:Measurement_Point_Round-SMD-Pad_Small" H 5250 2525 50  0001 C CNN
+F 3 "" H 5250 2525 50  0000 C CNN
+	1    5250 2525
+	-1   0    0    1
+$EndComp
+Wire Wire Line
+	5250 2525 5250 2520
+Connection ~ 5250 2520
 $EndSCHEMATC

Commit message: added tolerance
Parts:
- R14, R16: value 7k -> 7k 1%
- R15, R17: value 18k -> 18k 1%
- R18, R20: value 8k -> 8k 1%
- R19, R21: value 10.6k -> 10.6k 1%
- R8: value 18K -> 18K 1%
Changed lines of the file:
@@
 P 5290 4370
 F 0 "R8" V 5370 4370 50  0000 C CNN
-F 1 "18K" V 5290 4370 50  0000 C CNN
+F 1 "18K 1%" V 5290 4370 50  0000 C CNN
 F 2 "fdsp_resistor:R_1206_HandSoldering" V 5220 4370 50  0001 C CNN
 F 3 "" H 5290 4370 50  0001 C CNN
@@
 P 12430 6410
 F 0 "R14" V 12350 6530 50  0000 C CNN
-F 1 "7k" V 12430 6410 50  0000 C CNN
+F 1 "7k 1%" V 12430 6410 50  0000 C CNN
 F 2 "fdsp_resistor:R_1206_HandSoldering" V 12360 6410 30  0001 C CNN
 F 3 "" H 12430 6410 30  0000 C CNN
@@
 P 12730 6510
 F 0 "R18" V 12770 6670 42  0000 C CNN
-F 1 "8k" V 12730 6510 50  0000 C CNN
+F 1 "8k 1%" V 12730 6510 50  0000 C CNN
 F 2 "fdsp_resistor:R_1206_HandSoldering" H 12660 6510 30  0001 C CNN
 F 3 "" H 12730 6510 30  0000 C CNN
@@
 P 12430 6610
 F 0 "R15" V 12480 6430 50  0000 C CNN
-F 1 "18k" V 12430 6610 50  0000 C CNN
+F 1 "18k 1%" V 12430 6610 50  0000 C CNN
 F 2 "fdsp_resistor:R_1206_HandSoldering" V 12360 6610 30  0001 C CNN
 F 3 "" H 12430 6610 30  0000 C CNN
@@
 P 12730 6710
 F 0 "R19" V 12810 6710 50  0000 C CNN
-F 1 "10.6k" V 12730 6710 50  0000 C CNN
+F 1 "10.6k 1%" V 12730 6710 50  0000 C CNN
 F 2 "fdsp_resistor:R_1206_HandSoldering" V 12660 6710 30  0001 C CNN
 F 3 "" H 12730 6710 30  0000 C CNN
@@
 P 12470 7820
 F 0 "R16" V 12390 7940 50  0000 C CNN
-F 1 "7k" V 12470 7820 50  0000 C CNN
+F 1 "7k 1%" V 12470 7820 50  0000 C CNN
 F 2 "fdsp_resistor:R_1206_HandSoldering" V 12400 7820 30  0001 C CNN
 F 3 "" H 12470 7820 30  0000 C CNN
@@
 P 12770 7920
 F 0 "R20" V 12820 8090 50  0000 C CNN
-F 1 "8k" V 12770 7920 50  0000 C CNN
+F 1 "8k 1%" V 12770 7920 50  0000 C CNN
 F 2 "fdsp_resistor:R_1206_HandSoldering" H 12700 7920 30  0001 C CNN
 F 3 "" H 12770 7920 30  0000 C CNN
@@
 P 12470 8020
 F 0 "R17" V 12510 7840 50  0000 C CNN
-F 1 "18k" V 12470 8020 50  0000 C CNN
+F 1 "18k 1%" V 12470 8020 50  0000 C CNN
 F 2 "fdsp_resistor:R_1206_HandSoldering" V 12400 8020 30  0001 C CNN
 F 3 "" H 12470 8020 30  0000 C CNN
@@
 P 12770 8120
 F 0 "R21" V 12850 8120 50  0000 C CNN
-F 1 "10.6k" V 12770 8120 50  0000 C CNN
+F 1 "10.6k 1%" V 12770 8120 50  0000 C CNN
 F 2 "fdsp_resistor:R_1206_HandSoldering" V 12700 8120 30  0001 C CNN
 F 3 "" H 12770 8120 30  0000 C CNN

Commit message: kleine Anpassungen
Parts:
- C18: value 3n3 -> 3n3, <20%
- C19: value 56n -> 56n, <20%
- R10: value 475 -> 475, <10%
Changed lines of the file:
@@
 P 7360 2200
 F 0 "R10" V 7440 2200 50  0000 C CNN
-F 1 "475" V 7360 2200 50  0000 C CNN
+F 1 "475, <10%" V 7250 2150 50  0000 C CNN
 F 2 "fdsp_resistor:R_1206_HandSoldering" V 7290 2200 50  0001 C CNN
 F 3 "" H 7360 2200 50  0001 C CNN
@@
 P 6980 2620
 F 0 "C18" H 7005 2720 50  0000 L CNN
-F 1 "3n3" H 7005 2520 50  0000 L CNN
+F 1 "3n3, <20%" H 6800 2540 50  0000 L CNN
 F 2 "fdsp_capacitor:C_1206_HandSoldering" H 7018 2470 50  0001 C CNN
 F 3 "" H 6980 2620 50  0001 C CNN
@@
 P 7360 2620
 F 0 "C19" H 7385 2720 50  0000 L CNN
-F 1 "56n" H 7385 2520 50  0000 L CNN
+F 1 "56n, <20%" H 7385 2520 50  0000 L CNN
 F 2 "fdsp_capacitor:C_1206_HandSoldering" H 7398 2470 50  0001 C CNN
 F 3 "" H 7360 2620 50  0001 C CNN

Commit message: started layout
Parts:
- added P23: TST, fdsp_misc:Measurement_Point_Round-SMD-Pad_Small, symbol TST
Connections:
- net MP0: now also P23.1
Changed lines of the file:
@@
 Text GLabel 2650 2410 0    52   Input ~ 0
 MP1
-Text GLabel 2650 2310 0    52   Input ~ 0
+Text GLabel 2075 2310 0    52   Input ~ 0
 MP0
 $Comp
@@
 	5200 2320 5300 2320
 Wire Wire Line
-	5300 2520 5200 2520
+	5200 2520 5300 2520
 Wire Wire Line
 	7360 1920 7360 2050
@@
 	2650 2810 2720 2810
 Wire Wire Line
-	2720 2310 2650 2310
+	2720 2310 2075 2310
 Wire Wire Line
 	1990 6210 1990 5960
@@
 	5250 2525 5250 2520
 Connection ~ 5250 2520
+$Comp
+L TST P23
+U 1 1 5B240D5A
+P 2170 2270
+F 0 "P23" H 2170 2570 50  0000 C BNN
+F 1 "TST" H 2170 2520 50  0000 C CNN
+F 2 "fdsp_misc:Measurement_Point_Round-SMD-Pad_Small" H 2170 2270 50  0001 C CNN
+F 3 "" H 2170 2270 50  0000 C CNN
+	1    2170 2270
+	1    0    0    -1
+$EndComp
+Wire Wire Line
+	2170 2270 2170 2310
+Connection ~ 2170 2310
 $EndSCHEMATC
