File: SOURCES/smd_aio.sch (KiCad schematic (older format))
At the start: 64 parts, among them J1 RCA_01, J2 RCA_01, P1 CONN_01X06, P16 TST, P2 CONN_01X04, P23 TST, P3 CONN_01X03, P4 CONN_02X05, P5 STDCONN, P6 CONN_01X04, P7 CONN_02X04, P8 CONN_02X04, Q1 BSS123, Q2 BSS123, Q3 BSS123, Q4 BSS123, Q5 FZT751TA, SW1 SW_PUSH, U1 ADAU1701, U2 24AA256SN

Commit message: started layout
Parts:
- R6: value 1K -> 1K 1%
Changed lines of the file:
@@
 P 4080 1700
 F 0 "R6" V 4160 1700 50  0000 C CNN
-F 1 "1K" V 4080 1700 50  0000 C CNN
+F 1 "1K 1%" V 4080 1700 50  0000 C CNN
 F 2 "fdsp_resistor:R_1206_HandSoldering" V 4010 1700 50  0001 C CNN
 F 3 "" H 4080 1700 50  0001 C CNN

Commit message: layout, neue Clock Zuordnung
Connections:
- net MCLK3 renamed MCLK1
Changed lines of the file:
@@
 	7700 5880 7810 5880
 Text GLabel 7700 5980 0    52   Input ~ 0
-MCLK3
+MCLK1
 Wire Wire Line
 	7700 5980 7810 5980

Commit message: layout
Connections:
- net VIN: no longer D2.1 (K)
- new net VCC: D2.1 (K)
Changed lines of the file:
@@
 USBi Connector
-$Comp
-L VIN #PWR029
-U 1 1 5AFBD312
-P 5640 5340
-F 0 "#PWR029" H 5640 5190 50  0001 C CNN
-F 1 "VIN" H 5640 5480 50  0000 C CNN
-F 2 "" H 5640 5340 60  0000 C CNN
-F 3 "" H 5640 5340 60  0000 C CNN
-	1    5640 5340
-	1    0    0    -1
-$EndComp
 $Comp
 L CONN_01X03 P3
@@
 	2170 2270 2170 2310
 Connection ~ 2170 2310
+$Comp
+L VCC #PWR?
+U 1 1 5B2D3C23
+P 5640 5340
+F 0 "#PWR?" H 5640 5190 50  0001 C CNN
+F 1 "VCC" H 5640 5490 50  0000 C CNN
+F 2 "" H 5640 5340 60  0000 C CNN
+F 3 "" H 5640 5340 60  0000 C CNN
+	1    5640 5340
+	1    0    0    -1
+$EndComp
 $EndSCHEMATC

Commit message: layout
Parts:
- removed P6: CONN_01X04, fdsp_pinheader:Pin_Header_Straight_1x04, symbol CONN_01X04
- added P6: CONN_02X04, fdsp_pinheader:Pin_Header_Straight_2x04, symbol CONN_02X04
Connections:
- net GND: now also P6.2 (P2), P6.4 (P4), P6.6 (P6), P6.8 (P8)
- net VOUT0: now also P6.1 (P1)
- net VOUT1: now also P6.3 (P3)
- net VOUT2: now also P6.5 (P5)
- net VOUT3: now also P6.7 (P7)
Changed lines of the file:
@@
 Text GLabel 8940 7560 0    51   Input ~ 0
 VOUT3
-Text GLabel 8370 7740 0    55   Input ~ 0
-ADC1
-$Comp
-L CONN_01X04 P6
-U 1 1 5B050B23
-P 9180 7410
-F 0 "P6" H 9180 7660 50  0000 C CNN
-F 1 "CONN_01X04" V 9280 7410 50  0000 C CNN
-F 2 "fdsp_pinheader:Pin_Header_Straight_1x04" H 9180 7410 60  0001 C CNN
-F 3 "" H 9180 7410 60  0000 C CNN
-	1    9180 7410
-	1    0    0    -1
-$EndComp
 Wire Wire Line
 	8940 7260 8980 7260
@@
 	1    0    0    -1
 $EndComp
+$Comp
+L CONN_02X04 P6
+U 1 1 5B33B441
+P 9230 7410
+F 0 "P6" H 9230 7660 50  0000 C CNN
+F 1 "CONN_02X04" H 9230 7160 50  0000 C CNN
+F 2 "fdsp_pinheader:Pin_Header_Straight_2x04" H 9230 6210 60  0001 C CNN
+F 3 "" H 9230 6210 60  0000 C CNN
+	1    9230 7410
+	1    0    0    -1
+$EndComp
+$Comp
+L GND #PWR041
+U 1 1 5B33C668
+P 9525 7635
+F 0 "#PWR041" H 9525 7385 50  0001 C CNN
+F 1 "GND" H 9525 7485 50  0000 C CNN
+F 2 "" H 9525 7635 60  0000 C CNN
+F 3 "" H 9525 7635 60  0000 C CNN
+	1    9525 7635
+	1    0    0    -1
+$EndComp
+Wire Wire Line
+	9525 7260 9525 7635
+Wire Wire Line
+	9525 7560 9480 7560
+Wire Wire Line
+	9480 7460 9525 7460
+Connection ~ 9525 7560
+Wire Wire Line
+	9480 7360 9525 7360
+Connection ~ 9525 7460
+Wire Wire Line
+	9480 7260 9525 7260
+Connection ~ 9525 7360
 $EndSCHEMATC

Commit message: updated references
Parts:
- R19, R21: value 10.6k 1% -> 10k6 1%
Changed lines of the file:
@@
 P 12730 6710
 F 0 "R19" V 12810 6710 50  0000 C CNN
-F 1 "10.6k 1%" V 12730 6710 50  0000 C CNN
+F 1 "10k6 1%" V 12730 6710 50  0000 C CNN
 F 2 "fdsp_resistor:R_1206_HandSoldering" V 12660 6710 30  0001 C CNN
 F 3 "" H 12730 6710 30  0000 C CNN
@@
 P 12770 8120
 F 0 "R21" V 12850 8120 50  0000 C CNN
-F 1 "10.6k 1%" V 12770 8120 50  0000 C CNN
+F 1 "10k6 1%" V 12770 8120 50  0000 C CNN
 F 2 "fdsp_resistor:R_1206_HandSoldering" V 12700 8120 30  0001 C CNN
 F 3 "" H 12770 8120 30  0000 C CNN
