File: SOURCES/I2S-Amp2.sch (KiCad schematic (older format))
At the start: 33 parts, among them P14 CONN_01X02, P15 CONN_01X02, U8 SN74LVC14ADG4, U9 TAS5760MDCAR

Commit message: drc
Connections:
- no-connect marks 0 -> 17
Changed lines of the file:
@@
 Text GLabel 4050 3630 3    44   Input ~ 0
 MCLK2
+NoConn ~ 6450 3600
+NoConn ~ 6450 3700
+NoConn ~ 6450 3800
+NoConn ~ 6450 3900
+NoConn ~ 6450 4000
+NoConn ~ 6450 4100
+NoConn ~ 6450 4200
+NoConn ~ 5050 3600
+NoConn ~ 5050 3700
+NoConn ~ 5050 3800
+NoConn ~ 5050 3900
+NoConn ~ 5050 4000
+NoConn ~ 5050 4100
+NoConn ~ 5050 4200
+NoConn ~ 3050 2950
+NoConn ~ 3050 2750
+NoConn ~ 3050 3150
 $EndSCHEMATC

Commit message: finished drc
Parts:
- renumbered R37 to R39, R38 to R40, R39 to R41
Changed lines of the file:
@@
 $EndComp
 $Comp
-L GND #PWR0105
+L GND #PWR0113
 U 1 1 574C389A
 P 4450 1150
-F 0 "#PWR0105" H 4450 900 50  0001 C CNN
+F 0 "#PWR0113" H 4450 900 50  0001 C CNN
 F 1 "GND" H 4450 1000 50  0000 C CNN
 F 2 "" H 4450 1150 50  0000 C CNN
@@
 $EndComp
 $Comp
-L GND #PWR0106
+L GND #PWR0114
 U 1 1 574C3B84
 P 6600 2000
-F 0 "#PWR0106" H 6600 1750 50  0001 C CNN
+F 0 "#PWR0114" H 6600 1750 50  0001 C CNN
 F 1 "GND" H 6600 1850 50  0000 C CNN
 F 2 "" H 6600 2000 50  0000 C CNN
@@
 $EndComp
 $Comp
-L GND #PWR0107
+L GND #PWR0115
 U 1 1 574C3D2D
 P 7600 2100
-F 0 "#PWR0107" H 7600 1850 50  0001 C CNN
+F 0 "#PWR0115" H 7600 1850 50  0001 C CNN
 F 1 "GND" H 7600 1950 50  0000 C CNN
 F 2 "" H 7600 2100 50  0000 C CNN
@@
 $EndComp
 $Comp
-L GND #PWR0108
+L GND #PWR0116
 U 1 1 574C411D
 P 7050 1500
-F 0 "#PWR0108" H 7050 1250 50  0001 C CNN
+F 0 "#PWR0116" H 7050 1250 50  0001 C CNN
 F 1 "GND" H 7050 1350 50  0000 C CNN
 F 2 "" H 7050 1500 50  0000 C CNN
@@
 $EndComp
 $Comp
-L GND #PWR0109
+L GND #PWR0117
 U 1 1 574C436D
 P 3750 2850
-F 0 "#PWR0109" H 3750 2600 50  0001 C CNN
+F 0 "#PWR0117" H 3750 2600 50  0001 C CNN
 F 1 "GND" H 3750 2700 50  0000 C CNN
 F 2 "" H 3750 2850 50  0000 C CNN
@@
 $EndComp
 $Comp
-L GND #PWR0110
+L GND #PWR0118
 U 1 1 574C66FC
 P 6600 2600
-F 0 "#PWR0110" H 6600 2350 50  0001 C CNN
+F 0 "#PWR0118" H 6600 2350 50  0001 C CNN
 F 1 "GND" H 6600 2450 50  0000 C CNN
 F 2 "" H 6600 2600 50  0000 C CNN
@@
 $EndComp
 $Comp
-L GND #PWR0111
+L GND #PWR0119
 U 1 1 574C6724
 P 6600 3100
-F 0 "#PWR0111" H 6600 2850 50  0001 C CNN
+F 0 "#PWR0119" H 6600 2850 50  0001 C CNN
 F 1 "GND" H 6600 2950 50  0000 C CNN
 F 2 "" H 6600 3100 50  0000 C CNN
@@
 $EndComp
 $Comp
-L GND #PWR0112
+L GND #PWR0120
 U 1 1 574C7512
 P 7600 3700
-F 0 "#PWR0112" H 7600 3450 50  0001 C CNN
+F 0 "#PWR0120" H 7600 3450 50  0001 C CNN
 F 1 "GND" H 7600 3550 50  0000 C CNN
 F 2 "" H 7600 3700 50  0000 C CNN
@@
 $EndComp
 $Comp
-L GND #PWR0113
+L GND #PWR0121
 U 1 1 574CFB07
 P 9500 2350
-F 0 "#PWR0113" H 9500 2100 50  0001 C CNN
+F 0 "#PWR0121" H 9500 2100 50  0001 C CNN
 F 1 "GND" H 9500 2200 50  0000 C CNN
 F 2 "" H 9500 2350 50  0000 C CNN
@@
 $EndComp
 $Comp
-L GND #PWR0114
+L GND #PWR0122
 U 1 1 574CFB77
 P 9500 2850
-F 0 "#PWR0114" H 9500 2600 50  0001 C CNN
+F 0 "#PWR0122" H 9500 2600 50  0001 C CNN
 F 1 "GND" H 9500 2700 50  0000 C CNN
 F 2 "" H 9500 2850 50  0000 C CNN
@@
 $EndComp
 $Comp
-L GND #PWR0115
+L GND #PWR0123
 U 1 1 5B067D1E
 P 9500 3450
-F 0 "#PWR0115" H 9500 3200 50  0001 C CNN
+F 0 "#PWR0123" H 9500 3200 50  0001 C CNN
 F 1 "GND" H 9500 3300 50  0000 C CNN
 F 2 "" H 9500 3450 50  0000 C CNN
@@
 $EndComp
 $Comp
-L GND #PWR0116
+L GND #PWR0124
 U 1 1 5B067D1F
 P 9500 3950
-F 0 "#PWR0116" H 9500 3700 50  0001 C CNN
+F 0 "#PWR0124" H 9500 3700 50  0001 C CNN
 F 1 "GND" H 9500 3800 50  0000 C CNN
 F 2 "" H 9500 3950 50  0000 C CNN
@@
 $EndComp
 $Comp
-L GND #PWR0117
+L GND #PWR0125
 U 1 1 5750B753
 P 4900 3500
-F 0 "#PWR0117" H 4900 3250 50  0001 C CNN
+F 0 "#PWR0125" H 4900 3250 50  0001 C CNN
 F 1 "GND" H 4900 3350 50  0000 C CNN
 F 2 "" H 4900 3500 50  0000 C CNN
@@
 $EndComp
 $Comp
-L GND #PWR0118
+L GND #PWR0126
 U 1 1 5B067D26
 P 4900 2800
-F 0 "#PWR0118" H 4900 2550 50  0001 C CNN
+F 0 "#PWR0126" H 4900 2550 50  0001 C CNN
 F 1 "GND" H 4900 2650 50  0000 C CNN
 F 2 "" H 4900 2800 50  0000 C CNN
@@
 $EndComp
 $Comp
-L GND #PWR0119
+L GND #PWR0127
 U 1 1 5B067D27
 P 4900 2500
-F 0 "#PWR0119" H 4900 2250 50  0001 C CNN
+F 0 "#PWR0127" H 4900 2250 50  0001 C CNN
 F 1 "GND" H 4900 2350 50  0000 C CNN
 F 2 "" H 4900 2500 50  0000 C CNN
@@
 $EndComp
 $Comp
-L VCC #PWR0120
+L VCC #PWR0128
 U 1 1 5B067D2C
 P 8000 3400
-F 0 "#PWR0120" H 8000 3250 50  0001 C CNN
+F 0 "#PWR0128" H 8000 3250 50  0001 C CNN
 F 1 "VCC" H 8000 3550 50  0000 C CNN
 F 2 "" H 8000 3400 50  0000 C CNN
@@
 $EndComp
 $Comp
-L R R37
+L R R39
 U 1 1 575205B0
 P 1850 2000
-F 0 "R37" V 1930 2000 50  0000 C CNN
+F 0 "R39" V 1930 2000 50  0000 C CNN
 F 1 "100k" V 1850 2000 50  0000 C CNN
 F 2 "Resistors_SMD:R_0603" V 1780 2000 50  0001 C CNN
@@
 $EndComp
 $Comp
-L GND #PWR0121
+L GND #PWR0129
 U 1 1 5B067D2F
 P 1850 2400
-F 0 "#PWR0121" H 1850 2150 50  0001 C CNN
+F 0 "#PWR0129" H 1850 2150 50  0001 C CNN
 F 1 "GND" H 1850 2250 50  0000 C CNN
 F 2 "" H 1850 2400 50  0000 C CNN
@@
 $EndComp
 $Comp
-L GND #PWR0122
+L GND #PWR0130
 U 1 1 57526305
 P 1850 3250
-F 0 "#PWR0122" H 1850 3000 50  0001 C CNN
+F 0 "#PWR0130" H 1850 3000 50  0001 C CNN
 F 1 "GND" H 1850 3100 50  0000 C CNN
 F 2 "" H 1850 3250 50  0000 C CNN
@@
 $EndComp
 $Comp
-L GND #PWR0123
+L GND #PWR0131
 U 1 1 57542367
 P 2500 3150
-F 0 "#PWR0123" H 2500 2900 50  0001 C CNN
+F 0 "#PWR0131" H 2500 2900 50  0001 C CNN
 F 1 "GND" H 2500 3000 50  0000 C CNN
 F 2 "" H 2500 3150 50  0000 C CNN
@@
 $EndComp
 $Comp
-L VCC #PWR0124
+L VCC #PWR0132
 U 1 1 57556275
 P 8000 1800
-F 0 "#PWR0124" H 8000 1650 50  0001 C CNN
+F 0 "#PWR0132" H 8000 1650 50  0001 C CNN
 F 1 "VCC" H 8000 1950 50  0000 C CNN
 F 2 "" H 8000 1800 50  0000 C CNN
@@
 $EndComp
 $Comp
-L GND #PWR0125
+L GND #PWR0133
 U 1 1 5B067D2A
 P 3150 3150
-F 0 "#PWR0125" H 3150 2900 50  0001 C CNN
+F 0 "#PWR0133" H 3150 2900 50  0001 C CNN
 F 1 "GND" H 3150 3000 50  0000 C CNN
 F 2 "" H 3150 3150 50  0000 C CNN
@@
 $EndComp
 $Comp
-L R R39
+L R R41
 U 1 1 5B067D32
 P 3600 1850
-F 0 "R39" V 3680 1850 50  0000 C CNN
+F 0 "R41" V 3680 1850 50  0000 C CNN
 F 1 "120" V 3600 1850 50  0000 C CNN
 F 2 "Resistors_SMD:R_0603" V 3530 1850 50  0001 C CNN
@@
 $EndComp
 $Comp
-L R R38
+L R R40
 U 1 1 57531485
 P 1850 2850
-F 0 "R38" V 1930 2850 50  0000 C CNN
+F 0 "R40" V 1930 2850 50  0000 C CNN
 F 1 "100k" V 1850 2850 50  0000 C CNN
 F 2 "Resistors_SMD:R_0603" V 1780 2850 50  0001 C CNN
@@
 $EndComp
 $Comp
-L GND #PWR0126
+L GND #PWR0134
 U 1 1 575C07A8
 P 5750 4550
-F 0 "#PWR0126" H 5750 4300 50  0001 C CNN
+F 0 "#PWR0134" H 5750 4300 50  0001 C CNN
 F 1 "GND" H 5750 4400 50  0000 C CNN
 F 2 "" H 5750 4550 50  0000 C CNN
@@
 	4350 3400 4350 3630
 $Comp
-L +3V3 #PWR0127
+L +3V3 #PWR0135
 U 1 1 5AFA2E39
 P 1850 1770
-F 0 "#PWR0127" H 1850 1620 50  0001 C CNN
+F 0 "#PWR0135" H 1850 1620 50  0001 C CNN
 F 1 "+3V3" H 1850 1910 50  0000 C CNN
 F 2 "" H 1850 1770 60  0000 C CNN
@@
 $EndComp
 $Comp
-L +3V3 #PWR0128
+L +3V3 #PWR0136
 U 1 1 5AFA3723
 P 3600 1210
-F 0 "#PWR0128" H 3600 1060 50  0001 C CNN
+F 0 "#PWR0136" H 3600 1060 50  0001 C CNN
 F 1 "+3V3" H 3600 1350 50  0000 C CNN
 F 2 "" H 3600 1210 60  0000 C CNN
@@
 	3600 1210 3600 1300
 $Comp
-L +3V3 #PWR0129
+L +3V3 #PWR0137
 U 1 1 5B04DB98
 P 3350 2550
-F 0 "#PWR0129" H 3350 2400 50  0001 C CNN
+F 0 "#PWR0137" H 3350 2400 50  0001 C CNN
 F 1 "+3V3" H 3350 2690 50  0000 C CNN
 F 2 "" H 3350 2550 60  0000 C CNN
@@
 $EndComp
 $Comp
-L +3V3 #PWR0130
+L +3V3 #PWR0138
 U 1 1 5B067D4D
 P 3750 2600
-F 0 "#PWR0130" H 3750 2450 50  0001 C CNN
+F 0 "#PWR0138" H 3750 2450 50  0001 C CNN
 F 1 "+3V3" H 3750 2740 50  0000 C CNN
 F 2 "" H 3750 2600 60  0000 C CNN

Commit message: assign footprints
Parts:
- C69, C70, C72, C73, C74, C75, C76, C77, C80, C81, C82: footprint Capacitors_SMD:C_0603 -> fdsp_capacitor:C_1206_HandSoldering
- C71, C78, C79: value 0u1/35V -> 0u1/50V; footprint Capacitors_SMD:C_0603 -> fdsp_capacitor:C_1206_HandSoldering
- C83, C84: value 4u7/35V -> 4u7/50V; footprint Capacitors_SMD:C_1206 -> fdsp_capacitor:C_1206_HandSoldering
- C85, C86, C87, C88: value 0u68/35V -> 0u68/50V; footprint Capacitors_SMD:C_1206 -> fdsp_capacitor:C_1206_HandSoldering
- D9: footprint LEDs:LED_0603 -> fdsp_resistor:R_1206_HandSoldering
- L6, L7, L8, L9: footprint MyFootprints:1D10ASeries -> AMPx2 _footprints:1D10ASeries
- P14, P15: footprint MyFootprints:Connector0.5 -> (none)
- R37: renamed from R39; footprint Resistors_SMD:R_0603 -> fdsp_resistor:R_1206_HandSoldering
- R38: renamed from R40; footprint Resistors_SMD:R_0603 -> fdsp_resistor:R_1206_HandSoldering
- R39: renamed from R41; footprint Resistors_SMD:R_0603 -> fdsp_resistor:R_1206_HandSoldering
- RV2: footprint MyFootprints:M64Z104KB40 -> AMPx2 _footprints:M64Z104KB40
- U9: footprint MyFootprints:HTSSOP-48 -> AMPx2 _footprints:HTSSOP-48

Commit message: almost done footprints
Parts:
- P14, P15: footprint (none) -> fdsp_connector:RIACON101-2
Changed lines of the file:
@@
 F 0 "P15" H 10800 3550 50  0000 C CNN
 F 1 "CONN_01X02" V 10900 3400 50  0000 C CNN
-F 2 "" H 10800 3400 50  0001 C CNN
+F 2 "fdsp_connector:RIACON101-2" H 10800 3400 50  0001 C CNN
 F 3 "http://www.mouser.com/ds/2/324/ItemDetail_1935161-922578.pdf" H 10800 3400 50  0001 C CNN
 F 4 "1935161" H 10800 3400 60  0001 C CNN "Mfr.Nr."
@@
 F 0 "P14" H 10800 2450 50  0000 C CNN
 F 1 "CONN_01X02" V 10900 2300 50  0000 C CNN
-F 2 "" H 10800 2300 50  0001 C CNN
+F 2 "fdsp_connector:RIACON101-2" H 10800 2300 50  0001 C CNN
 F 3 "http://www.mouser.com/ds/2/324/ItemDetail_1935161-922578.pdf" H 10800 2300 50  0001 C CNN
 F 4 "1935161" H 10800 2300 60  0001 C CNN "Mfr.Nr."

Commit message: almost done footprints
Parts:
- added P21: TST, fdsp_misc:Measurement_Point_Round-SMD-Pad_Small, symbol TST
Connections:
- net MCLK2: now also P21.1
Changed lines of the file:
@@
 NoConn ~ 3050 2750
 NoConn ~ 3050 3150
+$Comp
+L TST P21
+U 1 1 5B2185A9
+P 4000 3550
+F 0 "P21" H 4000 3850 50  0000 C BNN
+F 1 "TST" H 4000 3800 50  0000 C CNN
+F 2 "fdsp_misc:Measurement_Point_Round-SMD-Pad_Small" H 4000 3550 50  0001 C CNN
+F 3 "" H 4000 3550 50  0000 C CNN
+	1    4000 3550
+	0    -1   -1   0
+$EndComp
+Wire Wire Line
+	4000 3550 4050 3550
+Connection ~ 4050 3550
 $EndSCHEMATC

Commit message: layout
Parts:
- C76, C80, C81, C82: footprint fdsp_capacitor:C_1206_HandSoldering -> fdsp_capacitor:C_0805_HandSoldering
Changed lines of the file:
@@
 F 0 "C80" V 7200 2500 50  0000 L CNN
 F 1 "0u22/25V" V 7200 2350 50  0000 R CNN
-F 2 "fdsp_capacitor:C_1206_HandSoldering" V 6850 2540 50  0001 C CNN
+F 2 "fdsp_capacitor:C_0805_HandSoldering" V 6850 2540 50  0001 C CNN
 F 3 "http://www.murata.com/products/catalog/pdf/c02e.pdf" V 6850 2540 50  0001 C CNN
 F 4 "GRM188R71E223KA01J" V 7150 2400 60  0001 C CNN "Mfr.Nr."
@@
 F 0 "C76" V 7050 2900 50  0000 L CNN
 F 1 "0u22/25V" V 7050 2750 50  0000 R CNN
-F 2 "fdsp_capacitor:C_1206_HandSoldering" V 6700 2940 50  0001 C CNN
+F 2 "fdsp_capacitor:C_0805_HandSoldering" V 6700 2940 50  0001 C CNN
 F 3 "http://www.murata.com/products/catalog/pdf/c02e.pdf" V 6700 2940 50  0001 C CNN
 F 4 "GRM188R71E223KA01J" V 7000 2800 60  0001 C CNN "Mfr.Nr."
@@
 F 0 "C82" V 7350 3000 50  0000 L CNN
 F 1 "0u22/25V" V 7350 2850 50  0000 R CNN
-F 2 "fdsp_capacitor:C_1206_HandSoldering" V 7000 3040 50  0001 C CNN
+F 2 "fdsp_capacitor:C_0805_HandSoldering" V 7000 3040 50  0001 C CNN
 F 3 "http://www.murata.com/products/catalog/pdf/c02e.pdf" V 7000 3040 50  0001 C CNN
 F 4 "GRM188R71E223KA01J" V 7300 2900 60  0001 C CNN "Mfr.Nr."
@@
 F 0 "C81" V 7200 3400 50  0000 L CNN
 F 1 "0u22/25V" V 7200 3250 50  0000 R CNN
-F 2 "fdsp_capacitor:C_1206_HandSoldering" V 6850 3440 50  0001 C CNN
+F 2 "fdsp_capacitor:C_0805_HandSoldering" V 6850 3440 50  0001 C CNN
 F 3 "http://www.murata.com/products/catalog/pdf/c02e.pdf" V 6850 3440 50  0001 C CNN
 F 4 "GRM188R71E223KA01J" V 7150 3300 60  0001 C CNN "Mfr.Nr."
