File: SOURCES/I2S-Amp2.sch (KiCad schematic (older format))
At the start: 34 parts, among them P14 CONN_01X02, P15 CONN_01X02, P21 TST, U8 SN74LVC14ADG4, U9 TAS5760MDCAR

Commit message: layout
Connections:
- net at C85.1, L6.2: now also P14.2 (P2); no longer P14.1 (P1)
- net at C86.1, L7.2: now also P14.1 (P1); no longer P14.2 (P2)
- net at C87.1, L8.2: now also P15.2 (P2); no longer P15.1 (P1)
- net at C88.1, L9.2: now also P15.1 (P1); no longer P15.2 (P2)
Other:
- moved on the sheet: P14, P15
Changed lines of the file:
@@
 L CONN_01X02 P15
 U 1 1 5B067D34
-P 10800 3400
-F 0 "P15" H 10800 3550 50  0000 C CNN
-F 1 "CONN_01X02" V 10900 3400 50  0000 C CNN
-F 2 "fdsp_connector:RIACON101-2" H 10800 3400 50  0001 C CNN
-F 3 "http://www.mouser.com/ds/2/324/ItemDetail_1935161-922578.pdf" H 10800 3400 50  0001 C CNN
-F 4 "1935161" H 10800 3400 60  0001 C CNN "Mfr.Nr."
-	1    10800 3400
-	1    0    0    -1
+P 10400 3400
+F 0 "P15" H 10400 3550 50  0000 C CNN
+F 1 "CONN_01X02" V 10500 3400 50  0000 C CNN
+F 2 "fdsp_connector:RIACON101-2" H 10400 3400 50  0001 C CNN
+F 3 "http://www.mouser.com/ds/2/324/ItemDetail_1935161-922578.pdf" H 10400 3400 50  0001 C CNN
+F 4 "1935161" H 10400 3400 60  0001 C CNN "Mfr.Nr."
+	1    10400 3400
+	-1   0    0    1
 $EndComp
 Text Label 4800 3100 0    60   ~ 0
@@
 L CONN_01X02 P14
 U 1 1 57584668
-P 10800 2300
-F 0 "P14" H 10800 2450 50  0000 C CNN
-F 1 "CONN_01X02" V 10900 2300 50  0000 C CNN
-F 2 "fdsp_connector:RIACON101-2" H 10800 2300 50  0001 C CNN
-F 3 "http://www.mouser.com/ds/2/324/ItemDetail_1935161-922578.pdf" H 10800 2300 50  0001 C CNN
-F 4 "1935161" H 10800 2300 60  0001 C CNN "Mfr.Nr."
-	1    10800 2300
-	1    0    0    -1
+P 10400 2300
+F 0 "P14" H 10400 2450 50  0000 C CNN
+F 1 "CONN_01X02" V 10500 2300 50  0000 C CNN
+F 2 "fdsp_connector:RIACON101-2" H 10400 2300 50  0001 C CNN
+F 3 "http://www.mouser.com/ds/2/324/ItemDetail_1935161-922578.pdf" H 10400 2300 50  0001 C CNN
+F 4 "1935161" H 10400 2300 60  0001 C CNN "Mfr.Nr."
+	1    10400 2300
+	-1   0    0    1
 $EndComp
 $Comp

Commit message: layout, neue Clock Zuordnung
Connections:
- net MCLK2 renamed MCLK5
Changed lines of the file:
@@
 MP11
 Text GLabel 4050 3630 3    44   Input ~ 0
-MCLK2
+MCLK5
 NoConn ~ 6450 3600
 NoConn ~ 6450 3700
