File: SOURCES/I2S-Amp1.sch (KiCad schematic (older format))
At the start: 33 parts, among them P10 CONN_01X02, P9 CONN_01X02, U3 SN74LVC14ADG4, U4 TAS5760MDCAR

Commit message: assign footprints
Parts:
- C22, C23, C25, C26, C27, C28, C29, C30, C33, C34, C35: footprint Capacitors_SMD:C_0603 -> fdsp_capacitor:C_1206_HandSoldering
- C24, C31, C32: value 0u1/35V -> 0u1/50V; footprint Capacitors_SMD:C_0603 -> fdsp_capacitor:C_1206_HandSoldering
- C36, C37: value 4u7/35V -> 4u7/50V; footprint Capacitors_SMD:C_1206 -> fdsp_capacitor:C_1206_HandSoldering
- C38, C39, C40, C41: value 0u68/35V -> 0u68/50V; footprint Capacitors_SMD:C_1206 -> fdsp_capacitor:C_1206_HandSoldering
- D3: footprint LEDs:LED_0603 -> fdsp_resistor:R_1206_HandSoldering
- L1, L2, L3, L4: footprint MyFootprints:1D10ASeries -> AMPx2 _footprints:1D10ASeries
- P10, P9: footprint MyFootprints:Connector0.5 -> (none)
- R22, R23, R24: footprint Resistors_SMD:R_0603 -> fdsp_resistor:R_1206_HandSoldering
- RV1: footprint MyFootprints:M64Z104KB40 -> AMPx2 _footprints:M64Z104KB40
- U4: footprint (none) -> AMPx2 _footprints:HTSSOP-48

Commit message: almost done footprints
Parts:
- P10, P9: footprint (none) -> fdsp_connector:RIACON101-2
Changed lines of the file:
@@
 F 0 "P10" H 10800 3550 50  0000 C CNN
 F 1 "CONN_01X02" V 10900 3400 50  0000 C CNN
-F 2 "" H 10800 3400 50  0001 C CNN
+F 2 "fdsp_connector:RIACON101-2" H 10800 3400 50  0001 C CNN
 F 3 "http://www.mouser.com/ds/2/324/ItemDetail_1935161-922578.pdf" H 10800 3400 50  0001 C CNN
 F 4 "1935161" H 10800 3400 60  0001 C CNN "Mfr.Nr."
@@
 F 0 "P9" H 10800 2450 50  0000 C CNN
 F 1 "CONN_01X02" V 10900 2300 50  0000 C CNN
-F 2 "" H 10800 2300 50  0001 C CNN
+F 2 "fdsp_connector:RIACON101-2" H 10800 2300 50  0001 C CNN
 F 3 "http://www.mouser.com/ds/2/324/ItemDetail_1935161-922578.pdf" H 10800 2300 50  0001 C CNN
 F 4 "1935161" H 10800 2300 60  0001 C CNN "Mfr.Nr."

Commit message: almost done footprints
Parts:
- added P17: TST, fdsp_misc:Measurement_Point_Round-SMD-Pad_Small, symbol TST
Connections:
- net MCLK1: now also P17.1
Changed lines of the file:
@@
 $EndComp
 NoConn ~ 6450 3600
+$Comp
+L TST P17
+U 1 1 5B216FDF
+P 4035 3520
+F 0 "P17" H 4035 3820 50  0000 C BNN
+F 1 "TST" H 4035 3770 50  0000 C CNN
+F 2 "fdsp_misc:Measurement_Point_Round-SMD-Pad_Small" H 4035 3520 50  0001 C CNN
+F 3 "" H 4035 3520 50  0000 C CNN
+	1    4035 3520
+	0    -1   -1   0
+$EndComp
+Wire Wire Line
+	4035 3520 4050 3520
+Connection ~ 4050 3520
 $EndSCHEMATC

Commit message: started layout
Parts:
- added P24, P25, P26: TST, fdsp_misc:Measurement_Point_Round-SMD-Pad_Small, symbol TST
Connections:
- net MP10: now also P26.1
- net MP11: now also P24.1
- net MP6: now also P25.1
Changed lines of the file:
@@
 	4050 3100 4050 3630
 Wire Wire Line
-	4150 3200 4150 3630
+	4150 3200 4150 4110
 Wire Wire Line
-	4250 3300 4250 3630
+	4250 3300 4250 4555
 Wire Wire Line
-	4350 3400 4350 3630
+	4350 3400 4350 3765
 $Comp
 L +3V3 #PWR063
@@
 	1    0    0    -1
 $EndComp
-Text GLabel 4350 3630 3    44   Input ~ 0
+Text GLabel 4350 3765 3    44   Input ~ 0
 MP10
-Text GLabel 4250 3630 3    44   Input ~ 0
+Text GLabel 4250 4555 3    44   Input ~ 0
 MP6
-Text GLabel 4150 3630 3    44   Input ~ 0
+Text GLabel 4150 4110 3    44   Input ~ 0
 MP11
 Text GLabel 4050 3630 3    44   Input ~ 0
@@
 	4035 3520 4050 3520
 Connection ~ 4050 3520
+$Comp
+L TST P24
+U 1 1 5B23E70D
+P 4130 4010
+F 0 "P24" H 4130 4310 50  0000 C BNN
+F 1 "TST" H 4130 4260 50  0000 C CNN
+F 2 "fdsp_misc:Measurement_Point_Round-SMD-Pad_Small" H 4130 4010 50  0001 C CNN
+F 3 "" H 4130 4010 50  0000 C CNN
+	1    4130 4010
+	0    -1   -1   0
+$EndComp
+Wire Wire Line
+	4130 4010 4150 4010
+Connection ~ 4150 4010
+$Comp
+L TST P25
+U 1 1 5B23EE58
+P 4215 4465
+F 0 "P25" H 4215 4765 50  0000 C BNN
+F 1 "TST" H 4215 4715 50  0000 C CNN
+F 2 "fdsp_misc:Measurement_Point_Round-SMD-Pad_Small" H 4215 4465 50  0001 C CNN
+F 3 "" H 4215 4465 50  0000 C CNN
+	1    4215 4465
+	0    -1   -1   0
+$EndComp
+Wire Wire Line
+	4215 4465 4250 4465
+Wire Wire Line
+	4250 4465 4250 4460
+Connection ~ 4250 4460
+$Comp
+L TST P26
+U 1 1 5B23F295
+P 4395 3690
+F 0 "P26" H 4395 3990 50  0000 C BNN
+F 1 "TST" H 4395 3940 50  0000 C CNN
+F 2 "fdsp_misc:Measurement_Point_Round-SMD-Pad_Small" H 4395 3690 50  0001 C CNN
+F 3 "" H 4395 3690 50  0000 C CNN
+	1    4395 3690
+	0    1    1    0
+$EndComp
+Wire Wire Line
+	4395 3690 4350 3690
+Connection ~ 4350 3690
 $EndSCHEMATC

Commit message: layout
Connections:
- net at C38.1, L1.2: now also P9.2 (P2); no longer P9.1 (P1)
- net at C40.1, L3.2: now also P10.2 (P2); no longer P10.1 (P1)
- net at C41.1, L4.2: now also P10.1 (P1); no longer P10.2 (P2)
- net at C39.1, L2.2: now also P9.1 (P1); no longer P9.2 (P2)
Other:
- moved on the sheet: P10, P9
Changed lines of the file:
@@
 L CONN_01X02 P10
 U 1 1 5753BEB1
-P 10800 3400
-F 0 "P10" H 10800 3550 50  0000 C CNN
-F 1 "CONN_01X02" V 10900 3400 50  0000 C CNN
-F 2 "fdsp_connector:RIACON101-2" H 10800 3400 50  0001 C CNN
-F 3 "http://www.mouser.com/ds/2/324/ItemDetail_1935161-922578.pdf" H 10800 3400 50  0001 C CNN
-F 4 "1935161" H 10800 3400 60  0001 C CNN "Mfr.Nr."
-	1    10800 3400
-	1    0    0    -1
+P 10400 3400
+F 0 "P10" H 10400 3550 50  0000 C CNN
+F 1 "CONN_01X02" V 10500 3400 50  0000 C CNN
+F 2 "fdsp_connector:RIACON101-2" H 10400 3400 50  0001 C CNN
+F 3 "http://www.mouser.com/ds/2/324/ItemDetail_1935161-922578.pdf" H 10400 3400 50  0001 C CNN
+F 4 "1935161" H 10400 3400 60  0001 C CNN "Mfr.Nr."
+	1    10400 3400
+	-1   0    0    1
 $EndComp
 Text Label 4800 3100 0    60   ~ 0
@@
 L CONN_01X02 P9
 U 1 1 5B067D3A
-P 10800 2300
-F 0 "P9" H 10800 2450 50  0000 C CNN
-F 1 "CONN_01X02" V 10900 2300 50  0000 C CNN
-F 2 "fdsp_connector:RIACON101-2" H 10800 2300 50  0001 C CNN
-F 3 "http://www.mouser.com/ds/2/324/ItemDetail_1935161-922578.pdf" H 10800 2300 50  0001 C CNN
-F 4 "1935161" H 10800 2300 60  0001 C CNN "Mfr.Nr."
-	1    10800 2300
-	1    0    0    -1
+P 10400 2300
+F 0 "P9" H 10400 2450 50  0000 C CNN
+F 1 "CONN_01X02" V 10500 2300 50  0000 C CNN
+F 2 "fdsp_connector:RIACON101-2" H 10400 2300 50  0001 C CNN
+F 3 "http://www.mouser.com/ds/2/324/ItemDetail_1935161-922578.pdf" H 10400 2300 50  0001 C CNN
+F 4 "1935161" H 10400 2300 60  0001 C CNN "Mfr.Nr."
+	1    10400 2300
+	-1   0    0    1
 $EndComp
 $Comp

Commit message: layout
Parts:
- C29, C33, C34, C35: footprint fdsp_capacitor:C_1206_HandSoldering -> fdsp_capacitor:C_0805_HandSoldering
Changed lines of the file:
@@
 F 0 "C33" V 7200 2500 50  0000 L CNN
 F 1 "0u22/25V" V 7200 2350 50  0000 R CNN
-F 2 "fdsp_capacitor:C_1206_HandSoldering" V 6850 2540 50  0001 C CNN
+F 2 "fdsp_capacitor:C_0805_HandSoldering" V 6850 2540 50  0001 C CNN
 F 3 "http://www.murata.com/products/catalog/pdf/c02e.pdf" V 6850 2540 50  0001 C CNN
 F 4 "GRM188R71E223KA01J" V 7150 2400 60  0001 C CNN "Mfr.Nr."
@@
 F 0 "C29" V 7050 2900 50  0000 L CNN
 F 1 "0u22/25V" V 7050 2750 50  0000 R CNN
-F 2 "fdsp_capacitor:C_1206_HandSoldering" V 6700 2940 50  0001 C CNN
+F 2 "fdsp_capacitor:C_0805_HandSoldering" V 6700 2940 50  0001 C CNN
 F 3 "http://www.murata.com/products/catalog/pdf/c02e.pdf" V 6700 2940 50  0001 C CNN
 F 4 "GRM188R71E223KA01J" V 7000 2800 60  0001 C CNN "Mfr.Nr."
@@
 F 0 "C35" V 7350 3000 50  0000 L CNN
 F 1 "0u22/25V" V 7350 2850 50  0000 R CNN
-F 2 "fdsp_capacitor:C_1206_HandSoldering" V 7000 3040 50  0001 C CNN
+F 2 "fdsp_capacitor:C_0805_HandSoldering" V 7000 3040 50  0001 C CNN
 F 3 "http://www.murata.com/products/catalog/pdf/c02e.pdf" V 7000 3040 50  0001 C CNN
 F 4 "GRM188R71E223KA01J" V 7300 2900 60  0001 C CNN "Mfr.Nr."
@@
 F 0 "C34" V 7200 3400 50  0000 L CNN
 F 1 "0u22/25V" V 7200 3250 50  0000 R CNN
-F 2 "fdsp_capacitor:C_1206_HandSoldering" V 6850 3440 50  0001 C CNN
+F 2 "fdsp_capacitor:C_0805_HandSoldering" V 6850 3440 50  0001 C CNN
 F 3 "http://www.murata.com/products/catalog/pdf/c02e.pdf" V 6850 3440 50  0001 C CNN
 F 4 "GRM188R71E223KA01J" V 7150 3300 60  0001 C CNN "Mfr.Nr."

Commit message: layout, neue Clock Zuordnung
Connections:
- net MCLK1 renamed MCLK4
Changed lines of the file:
@@
 MP11
 Text GLabel 4050 3630 3    44   Input ~ 0
-MCLK1
+MCLK4
 NoConn ~ 5050 3600
 NoConn ~ 5050 3700
